Commit message: 2 links

File: body.urdf (robot description, URDF)
Before this commit: robot robot, 2 links, 1 joints
Links:
- removed link Leg
- removed link Torso
- added link Link0, mass 1; collision box size=1.0 1.0 1.0; visual box size=1.0 1.0 1.0
- added link Link1, mass 1; collision box size=1 1 1; visual box size=1 1 1
Joints:
- removed joint Torso_Leg
- added joint Link0_Link1: type revolute, parent Link0, child Link1, origin xyz=0.0 0.0 1.0 rpy=0 0 0, axis 0 1 0, limit lower=-3.14159 upper=3.14159 effort=0.0 velocity=0.0

Commit message: 3 links

File: body.urdf (robot description, URDF)
Before this commit: robot robot, 2 links, 1 joints
Links:
- added link Link2, mass 1; collision box size=1 1 1; visual box size=1 1 1
Joints:
- added joint Link1_Link2: type revolute, parent Link1, child Link2, origin xyz=0.0 0.0 1.0 rpy=0 0 0, axis 0 1 0, limit lower=-3.14159 upper=3.14159 effort=0.0 velocity=0.0

Commit message: 4 links

File: body.urdf (robot description, URDF)
Before this commit: robot robot, 3 links, 2 joints
Links:
- added link Link3, mass 1; collision box size=1 1 1; visual box size=1 1 1
Joints:
- added joint Link2_Link3: type revolute, parent Link2, child Link3, origin xyz=0.0 0.5 0.5 rpy=0 0 0, axis 0 1 0, limit lower=-3.14159 upper=3.14159 effort=0.0 velocity=0.0

Commit message: 5 links

File: body.urdf (robot description, URDF)
Before this commit: robot robot, 4 links, 3 joints
Links:
- added link Link4, mass 1; collision box size=1 1 1; visual box size=1 1 1
Joints:
- added joint Link3_Link4: type revolute, parent Link3, child Link4, origin xyz=0.0 1.0 0.0 rpy=0 0 0, axis 0 1 0, limit lower=-3.14159 upper=3.14159 effort=0.0 velocity=0.0

Commit message: torso and back leg work well

File: body.urdf (robot description, URDF)
Before this commit: robot robot, 5 links, 4 joints
Links:
- removed link Link0
- removed link Link1
- removed link Link2
- removed link Link3
- removed link Link4
- added link Back_Leg, mass 1; collision box size=1 1 1; visual box size=1 1 1
- added link Torso, mass 1; collision box size=1.0 1.0 1.0; visual box size=1.0 1.0 1.0
Joints:
- removed joint Link0_Link1
- removed joint Link1_Link2
- removed joint Link2_Link3
- removed joint Link3_Link4
- added joint Torso_Back_Leg: type revolute, parent Torso, child Back_Leg, origin xyz=1.0 0.0 1.0 rpy=0 0 0, axis 0 1 0, limit lower=-3.14159 upper=3.14159 effort=0.0 velocity=0.0

Commit message: working on front leg

File: body.urdf (robot description, URDF)
Before this commit: robot robot, 2 links, 1 joints
Links:
- added link Front_Leg, mass 1; collision box size=1 1 1; visual box size=1 1 1
Joints:
- added joint Torso_Front_Leg: type revolute, parent Torso, child Front_Leg, origin xyz=1.0 0.0 0.0 rpy=0 0 0, axis 0 1 0, limit lower=-3.14159 upper=3.14159 effort=0.0 velocity=0.0

Commit message: torso and legs added

File: body.urdf (robot description, URDF)
Before this commit: robot robot, 3 links, 2 joints
Links:
- removed link Back_Leg
- removed link Front_Leg
- added link BackLeg, mass 1; collision box size=1 1 1; visual box size=1 1 1
- added link FrontLeg, mass 1; collision box size=1 1 1; visual box size=1 1 1
Joints:
- removed joint Torso_Back_Leg
- removed joint Torso_Front_Leg
- added joint Torso_BackLeg: type revolute, parent Torso, child BackLeg, origin xyz=1.0 0.0 1.0 rpy=0 0 0, axis 0 1 0, limit lower=-3.14159 upper=3.14159 effort=0.0 velocity=0.0
- added joint Torso_FrontLeg: type revolute, parent Torso, child FrontLeg, origin xyz=1.0 0.0 0.0 rpy=0 0 0, axis 0 1 0, limit lower=-3.14159 upper=3.14159 effort=0.0 velocity=0.0

Commit message: fixed hinge joint for left leg

File: body.urdf (robot description, URDF)
Before this commit: robot robot, 3 links, 2 joints
Joints:
- joint Torso_FrontLeg: origin xyz=1.0 0.0 0.0 rpy=0 0 0 -> xyz=2.0 0.0 1.0 rpy=0 0 0

Commit message: front leg section complete

File: body.urdf (robot description, URDF)
Before this commit: robot robot, 3 links, 2 joints
Links:
- link FrontLeg: geometry collision box size=0.2 1 0.2; visual box size=0.2 1 0.2
Joints:
- joint Torso_FrontLeg: origin xyz=2.0 0.0 1.0 rpy=0 0 0 -> xyz=0.0 0.5 1.0 rpy=0 0 0

Commit message: back leg is added

File: body.urdf (robot description, URDF)
Before this commit: robot robot, 3 links, 2 joints
Links:
- link BackLeg: geometry collision box size=0.2 1 0.2; visual box size=0.2 1 0.2
Joints:
- joint Torso_BackLeg: origin xyz=1.0 0.0 1.0 rpy=0 0 0 -> xyz=0.0 -0.5 1.0 rpy=0 0 0

Commit message: all 4 top legs added

File: body.urdf (robot description, URDF)
Before this commit: robot robot, 3 links, 2 joints
Links:
- added link LeftLeg, mass 1; collision box size=1 0.2 0.2; visual box size=1 0.2 0.2
- added link RightLeg, mass 1; collision box size=1 0.2 0.2; visual box size=1 0.2 0.2
Joints:
- added joint Torso_LeftLeg: type revolute, parent Torso, child LeftLeg, origin xyz=-0.5 0.0 1.0 rpy=0 0 0, axis 1 0 0, limit lower=-3.14159 upper=3.14159 effort=0.0 velocity=0.0
- added joint Torso_RightLeg: type revolute, parent Torso, child RightLeg, origin xyz=0.5 0.0 1.0 rpy=0 0 0, axis 1 0 0, limit lower=-3.14159 upper=3.14159 effort=0.0 velocity=0.0

Commit message: added all 4 legs, seems off

File: body.urdf (robot description, URDF)
Before this commit: robot robot, 5 links, 4 joints
Links:
- added link BackLowerLeg, mass 1; collision box size=0.2 0.2 1; visual box size=0.2 0.2 1
- added link FrontLowerLeg, mass 1; collision box size=0.2 0.2 1; visual box size=0.2 0.2 1
- added link LeftLowerLeg, mass 1; collision box size=0.2 0.2 1; visual box size=0.2 0.2 1
- added link RightLowerLeg, mass 1; collision box size=0.2 0.2 1; visual box size=0.2 0.2 1
Joints:
- added joint Torso_BackLowerLeg: type revolute, parent Torso, child BackLowerLeg, origin xyz=0.0 -1.0 0.0 rpy=0 0 0, axis 1 0 0, limit lower=-3.14159 upper=3.14159 effort=0.0 velocity=0.0
- added joint Torso_FrontLowerLeg: type revolute, parent Torso, child FrontLowerLeg, origin xyz=0.0 1.0 0.0 rpy=0 0 0, axis 1 0 0, limit lower=-3.14159 upper=3.14159 effort=0.0 velocity=0.0
- added joint Torso_LeftLowerLeg: type revolute, parent Torso, child LeftLowerLeg, origin xyz=-1.0 0.0 0.0 rpy=0 0 0, axis 1 0 0, limit lower=-3.14159 upper=3.14159 effort=0.0 velocity=0.0
- added joint Torso_RightLowerLeg: type revolute, parent Torso, child RightLowerLeg, origin xyz=1.0 0.0 0.0 rpy=0 0 0, axis 1 0 0, limit lower=-3.14159 upper=3.14159 effort=0.0 velocity=0.0

Commit message: fixed quadruped's leg positions, had the wrong parent

File: body.urdf (robot description, URDF)
Before this commit: robot robot, 9 links, 8 joints
Joints:
- joint Torso_BackLowerLeg: parent Torso -> BackLeg
- joint Torso_FrontLowerLeg: parent Torso -> FrontLeg
- joint Torso_LeftLowerLeg: parent Torso -> LeftLeg
- joint Torso_RightLowerLeg: parent Torso -> RightLeg

Commit message: fixed select

File: body.urdf (robot description, URDF)
Before this commit: robot robot, 9 links, 8 joints
Joints:
- joint Torso_LeftLowerLeg: axis 1 0 0 -> 0 1 0
- joint Torso_RightLowerLeg: axis 1 0 0 -> 0 1 0

Commit message: done with quadruped, part N

File: body.urdf (robot description, URDF)
Before this commit: robot robot, 9 links, 8 joints
Joints:
- joint Torso_BackLeg: axis 1 0 0 -> 0 1 0
- joint Torso_BackLowerLeg: axis 1 0 0 -> 0 1 0
- joint Torso_FrontLeg: axis 1 0 0 -> 0 1 0
- joint Torso_FrontLowerLeg: axis 1 0 0 -> 0 1 0
- joint Torso_LeftLeg: axis 1 0 0 -> 0 1 0
- joint Torso_RightLeg: axis 1 0 0 -> 0 1 0

Commit message: added extra robot legs with prismatic sliders

File: body.urdf (robot description, URDF)
Before this commit: robot robot, 9 links, 8 joints
Links:
- added link BackLowerLowerLeg, mass 1; collision box size=0.2 0.2 1; visual box size=0.2 0.2 1
- added link FrontLowerLowerLeg, mass 1; collision box size=0.2 0.2 1; visual box size=0.2 0.2 1
- added link LeftLowerLowerLeg, mass 1; collision box size=0.2 0.2 1; visual box size=0.2 0.2 1
- added link RightLowerLowerLeg, mass 1; collision box size=0.2 0.2 1; visual box size=0.2 0.2 1
Joints:
- added joint Lower_BackLowerLeg: type prismatic, parent BackLowerLeg, child BackLowerLowerLeg, origin xyz=0.0 0.0 -1.0 rpy=0 0 0, axis 0 0 1, limit lower=-3.14159 upper=3.14159 effort=0.0 velocity=0.0
- added joint Lower_FrontLowerLeg: type prismatic, parent FrontLowerLeg, child FrontLowerLowerLeg, origin xyz=0.0 0.0 -1.0 rpy=0 0 0, axis 0 0 1, limit lower=-3.14159 upper=3.14159 effort=0.0 velocity=0.0
- added joint Lower_LeftLowerLeg: type prismatic, parent LeftLowerLeg, child LeftLowerLowerLeg, origin xyz=0.0 0.0 -1.0 rpy=0 0 0, axis 0 0 1, limit lower=-3.14159 upper=3.14159 effort=0.0 velocity=0.0
- added joint Lower_RightLowerLeg: type prismatic, parent RightLowerLeg, child RightLowerLowerLeg, origin xyz=0.0 0.0 -1.0 rpy=0 0 0, axis 0 0 1, limit lower=-3.14159 upper=3.14159 effort=0.0 velocity=0.0
- joint Torso_BackLeg: origin xyz=0.0 -0.5 1.0 rpy=0 0 0 -> xyz=0.0 -0.5 2.0 rpy=0 0 0
- joint Torso_FrontLeg: origin xyz=0.0 0.5 1.0 rpy=0 0 0 -> xyz=0.0 0.5 2.0 rpy=0 0 0
- joint Torso_LeftLeg: origin xyz=-0.5 0.0 1.0 rpy=0 0 0 -> xyz=-0.5 0.0 2.0 rpy=0 0 0
- joint Torso_RightLeg: origin xyz=0.5 0.0 1.0 rpy=0 0 0 -> xyz=0.5 0.0 2.0 rpy=0 0 0

Commit message: legs slightly offset properly

File: body.urdf (robot description, URDF)
Before this commit: robot robot, 13 links, 12 joints
Joints:
- joint Torso_BackLeg: origin xyz=0.0 -0.5 2.0 rpy=0 0 0 -> xyz=0.25 -0.5 2.0 rpy=0 0 0
- joint Torso_FrontLeg: origin xyz=0.0 0.5 2.0 rpy=0 0 0 -> xyz=0.25 0.5 2.0 rpy=0 0 0
- joint Torso_LeftLeg: origin xyz=-0.5 0.0 2.0 rpy=0 0 0 -> xyz=-0.5 0.25 2.0 rpy=0 0 0
- joint Torso_RightLeg: origin xyz=0.5 0.0 2.0 rpy=0 0 0 -> xyz=0.5 0.25 2.0 rpy=0 0 0

Commit message: 8 legs added

File: body.urdf (robot description, URDF)
Before this commit: robot robot, 13 links, 12 joints
Links:
- added link BackSideLeg, mass 1; collision box size=0.2 1 0.2; visual box size=0.2 1 0.2
- added link BackSideLowerLeg, mass 1; collision box size=0.2 0.2 1; visual box size=0.2 0.2 1
- added link BackSideLowerLowerLeg, mass 1; collision box size=0.2 0.2 1; visual box size=0.2 0.2 1
- added link FrontSideLeg, mass 1; collision box size=0.2 1 0.2; visual box size=0.2 1 0.2
- added link FrontSideLowerLeg, mass 1; collision box size=0.2 0.2 1; visual box size=0.2 0.2 1
- added link FrontSideLowerLowerLeg, mass 1; collision box size=0.2 0.2 1; visual box size=0.2 0.2 1
- added link LeftSideLeg, mass 1; collision box size=1 0.2 0.2; visual box size=1 0.2 0.2
- added link LeftSideLowerLeg, mass 1; collision box size=0.2 0.2 1; visual box size=0.2 0.2 1
- added link LeftSideLowerLowerLeg, mass 1; collision box size=0.2 0.2 1; visual box size=0.2 0.2 1
- added link RightSideLeg, mass 1; collision box size=1 0.2 0.2; visual box size=1 0.2 0.2
- added link RightSideLowerLeg, mass 1; collision box size=0.2 0.2 1; visual box size=0.2 0.2 1
- added link RightSideLowerLowerLeg, mass 1; collision box size=0.2 0.2 1; visual box size=0.2 0.2 1
Joints:
- added joint Lower_BackSideLowerLeg: type prismatic, parent BackSideLowerLeg, child BackSideLowerLowerLeg, origin xyz=0.0 0.0 -1.0 rpy=0 0 0, axis 0 0 1, limit lower=-3.14159 upper=3.14159 effort=0.0 velocity=0.0
- added joint Lower_FrontSideLowerLeg: type prismatic, parent FrontSideLowerLeg, child FrontSideLowerLowerLeg, origin xyz=0.0 0.0 -1.0 rpy=0 0 0, axis 0 0 1, limit lower=-3.14159 upper=3.14159 effort=0.0 velocity=0.0
- added joint Lower_LeftSideLowerLeg: type prismatic, parent LeftSideLowerLeg, child LeftSideLowerLowerLeg, origin xyz=0.0 0.0 -1.0 rpy=0 0 0, axis 0 0 1, limit lower=-3.14159 upper=3.14159 effort=0.0 velocity=0.0
- added joint Lower_RightSideLowerLeg: type prismatic, parent RightSideLowerLeg, child RightSideLowerLowerLeg, origin xyz=0.0 0.0 -1.0 rpy=0 0 0, axis 0 0 1, limit lower=-3.14159 upper=3.14159 effort=0.0 velocity=0.0
- added joint Torso_BackSideLeg: type revolute, parent Torso, child BackSideLeg, origin xyz=-0.25 -0.5 2.0 rpy=0 0 0, axis 0 1 0, limit lower=-3.14159 upper=3.14159 effort=0.0 velocity=0.0
- added joint Torso_BackSideLowerLeg: type revolute, parent BackSideLeg, child BackSideLowerLeg, origin xyz=0.0 -1.0 0.0 rpy=0 0 0, axis 0 1 0, limit lower=-3.14159 upper=3.14159 effort=0.0 velocity=0.0
- added joint Torso_FrontSideLeg: type revolute, parent Torso, child FrontSideLeg, origin xyz=-0.25 0.5 2.0 rpy=0 0 0, axis 0 1 0, limit lower=-3.14159 upper=3.14159 effort=0.0 velocity=0.0
- added joint Torso_FrontSideLowerLeg: type revolute, parent FrontSideLeg, child FrontSideLowerLeg, origin xyz=0.0 1.0 0.0 rpy=0 0 0, axis 0 1 0, limit lower=-3.14159 upper=3.14159 effort=0.0 velocity=0.0
- added joint Torso_LeftSideLeg: type revolute, parent Torso, child LeftSideLeg, origin xyz=-0.5 -0.25 2.0 rpy=0 0 0, axis 0 1 0, limit lower=-3.14159 upper=3.14159 effort=0.0 velocity=0.0
- added joint Torso_LeftSideLowerLeg: type revolute, parent LeftSideLeg, child LeftSideLowerLeg, origin xyz=-1.0 0.0 0.0 rpy=0 0 0, axis 0 1 0, limit lower=-3.14159 upper=3.14159 effort=0.0 velocity=0.0
- added joint Torso_RightSideLeg: type revolute, parent Torso, child RightSideLeg, origin xyz=0.5 -0.25 2.0 rpy=0 0 0, axis 0 1 0, limit lower=-3.14159 upper=3.14159 effort=0.0 velocity=0.0
- added joint Torso_RightSideLowerLeg: type revolute, parent RightSideLeg, child RightSideLowerLeg, origin xyz=1.0 0.0 0.0 rpy=0 0 0, axis 0 1 0, limit lower=-3.14159 upper=3.14159 effort=0.0 velocity=0.0

Commit message: going to check previous checkpoint

File: body.urdf (robot description, URDF)
Before this commit: robot robot, 25 links, 24 joints
Links:
- added link Box, mass 1; collision box size=0.5 0.5 0.5; visual box size=0.5 0.5 0.5
Joints:
- added joint Torso_Box: type spherical, parent Torso, child Box, origin xyz=0.0 0 2.0 rpy=0 0 0, axis 0 1 0, limit lower=-3.14159 upper=3.14159 effort=0.0 velocity=0.0
- joint Lower_BackLowerLeg: axis 0 0 1 -> 0 1 0; type prismatic -> revolute
- joint Lower_BackSideLowerLeg: axis 0 0 1 -> 0 1 0; type prismatic -> revolute
- joint Lower_FrontLowerLeg: axis 0 0 1 -> 0 1 0; type prismatic -> revolute
- joint Lower_FrontSideLowerLeg: axis 0 0 1 -> 0 1 0; type prismatic -> revolute
- joint Lower_LeftLowerLeg: axis 0 0 1 -> 0 1 0; type prismatic -> revolute
- joint Lower_LeftSideLowerLeg: axis 0 0 1 -> 0 1 0; type prismatic -> revolute
- joint Lower_RightLowerLeg: axis 0 0 1 -> 0 1 0; type prismatic -> revolute
- joint Lower_RightSideLowerLeg: axis 0 0 1 -> 0 1 0; type prismatic -> revolute

Commit message: switching branches again

File: body.urdf (robot description, URDF)
Before this commit: robot robot, 26 links, 25 joints
Links:
- removed link BackLowerLowerLeg
- removed link BackSideLowerLowerLeg
- removed link FrontLowerLowerLeg
- removed link FrontSideLowerLowerLeg
- removed link LeftLowerLowerLeg
- removed link LeftSideLowerLowerLeg
- removed link RightLowerLowerLeg
- removed link RightSideLowerLowerLeg
Joints:
- removed joint Lower_BackLowerLeg
- removed joint Lower_BackSideLowerLeg
- removed joint Lower_FrontLowerLeg
- removed joint Lower_FrontSideLowerLeg
- removed joint Lower_LeftLowerLeg
- removed joint Lower_LeftSideLowerLeg
- removed joint Lower_RightLowerLeg
- removed joint Lower_RightSideLowerLeg

Commit message: reverted to quadruped

File: body.urdf (robot description, URDF)
Before this commit: robot robot, 18 links, 17 joints
Links:
- removed link BackSideLeg
- removed link BackSideLowerLeg
- removed link Box
- removed link FrontSideLeg
- removed link FrontSideLowerLeg
- removed link LeftSideLeg
- removed link LeftSideLowerLeg
- removed link RightSideLeg
- removed link RightSideLowerLeg
Joints:
- removed joint Torso_BackSideLeg
- removed joint Torso_BackSideLowerLeg
- removed joint Torso_Box
- removed joint Torso_FrontSideLeg
- removed joint Torso_FrontSideLowerLeg
- removed joint Torso_LeftSideLeg
- removed joint Torso_LeftSideLowerLeg
- removed joint Torso_RightSideLeg
- removed joint Torso_RightSideLowerLeg
- joint Torso_BackLeg: origin xyz=0.25 -0.5 2.0 rpy=0 0 0 -> xyz=0.0 -0.5 1.0 rpy=0 0 0
- joint Torso_FrontLeg: origin xyz=0.25 0.5 2.0 rpy=0 0 0 -> xyz=0.0 0.5 1.0 rpy=0 0 0
- joint Torso_LeftLeg: origin xyz=-0.5 0.25 2.0 rpy=0 0 0 -> xyz=-0.5 0.0 1.0 rpy=0 0 0
- joint Torso_RightLeg: origin xyz=0.5 0.25 2.0 rpy=0 0 0 -> xyz=0.5 0.0 1.0 rpy=0 0 0

Commit message: going to change the fitness function now

File: body.urdf (robot description, URDF)
Before this commit: robot robot, 9 links, 8 joints
Links:
- added link HittingLeg, mass 1; collision box size=0.2 0.2 1; visual box size=0.2 0.2 1
Joints:
- added joint Torso_HittingLeg: type revolute, parent Torso, child HittingLeg, origin xyz=0.0 0.0 1.0 rpy=0 0 0, axis 0 1 0, limit lower=-3.14159 upper=3.14159 effort=0.0 velocity=0.0

Commit message: done with final project

File: body.urdf (robot description, URDF)
Before this commit: robot robot, 10 links, 9 joints
Links:
- link BackLowerLeg: geometry collision box size=0.2 0.8 1; visual box size=0.2 0.8 1
- link FrontLowerLeg: geometry collision box size=0.2 0.8 1; visual box size=0.2 0.8 1
- link LeftLowerLeg: geometry collision box size=0.2 0.8 1; visual box size=0.2 0.8 1
- link RightLowerLeg: geometry collision box size=0.2 0.8 1; visual box size=0.2 0.8 1
Joints:
- joint Torso_HittingLeg: origin xyz=0.0 0.0 1.0 rpy=0 0 0 -> xyz=0.0 0.0 1.5 rpy=0 0 0

Commit message: code for 1 cube working but debugging for multiple

File: body.urdf (robot description, URDF)
Before this commit: robot robot, 10 links, 9 joints
Links:
- removed link BackLeg
- removed link BackLowerLeg
- removed link FrontLeg
- removed link FrontLowerLeg
- removed link HittingLeg
- removed link LeftLeg
- removed link LeftLowerLeg
- removed link RightLeg
- removed link RightLowerLeg
- removed link Torso
- added link Cube0, mass 1; collision box size=2.7764480012439217 2.2812546462312335 0.9096863272166162; visual box size=2.7764480012439217 2.2812546462312335 0.9096863272166162
- added link Cube1, mass 1; collision box size=2.354523666422527 1.5801956637886003 0.7890100203593798; visual box size=2.354523666422527 1.5801956637886003 0.7890100203593798
- added link Cube2, mass 1; collision box size=2.069809026158155 2.957738162305494 1.816563005656393; visual box size=2.069809026158155 2.957738162305494 1.816563005656393
- added link Cube3, mass 1; collision box size=0.5033335816554969 0.6354124277528632 0.8172234999852188; visual box size=0.5033335816554969 0.6354124277528632 0.8172234999852188
- added link Cube4, mass 1; collision box size=1.4724479017262602 0.5771326004338452 1.414655729657721; visual box size=1.4724479017262602 0.5771326004338452 1.414655729657721
- added link Cube5, mass 1; collision box size=1.4733950285711512 0.835568208310052 1.9373320096331885; visual box size=1.4733950285711512 0.835568208310052 1.9373320096331885
- added link Cube6, mass 1; collision box size=2.1131710043596525 0.6268460126145463 2.456771768773762; visual box size=2.1131710043596525 0.6268460126145463 2.456771768773762
- added link Cube7, mass 1; collision box size=0.8670453615297351 1.5713626757839565 1.7598872763889304; visual box size=0.8670453615297351 1.5713626757839565 1.7598872763889304
Joints:
- removed joint Torso_BackLeg
- removed joint Torso_BackLowerLeg
- removed joint Torso_FrontLeg
- removed joint Torso_FrontLowerLeg
- removed joint Torso_HittingLeg
- removed joint Torso_LeftLeg
- removed joint Torso_LeftLowerLeg
- removed joint Torso_RightLeg
- removed joint Torso_RightLowerLeg
- added joint jointName: type revolute, parent prevStringName, child stringName, origin xyz=0.0 0.31342300630727316 1.228385884386881 rpy=0 0 0, axis 0 1 0, limit lower=-3.14159 upper=3.14159 effort=0.0 velocity=0.0

Commit message: creates correct number of links, need to fix where they join

File: body.urdf (robot description, URDF)
Before this commit: robot robot, 8 links, 1 joints
Links:
- removed link Cube2
- removed link Cube3
- removed link Cube4
- removed link Cube5
- removed link Cube6
- removed link Cube7
- link Cube0: geometry collision box size=0.6424922441688098 1.8552213454617767 2.713225695080267; visual box size=0.6424922441688098 1.8552213454617767 2.713225695080267
- link Cube1: geometry collision box size=2.5127803270796942 1.207547853623944 2.7968453845835253; visual box size=2.5127803270796942 1.207547853623944 2.7968453845835253
Joints:
- removed joint jointName
- added joint Cube0_Cube1: type revolute, parent Cube0, child Cube1, origin xyz=0.0 0.9276106727308884 1.3566128475401336 rpy=0 0 0, axis 0 1 0, limit lower=-3.14159 upper=3.14159 effort=0.0 velocity=0.0

Commit message: joints work with 2 links

File: body.urdf (robot description, URDF)
Before this commit: robot robot, 2 links, 1 joints
Links:
- link Cube0: geometry collision box size=0.5668012223169285 1.1625662692443939 1.7872907515699616; visual box size=0.5668012223169285 1.1625662692443939 1.7872907515699616
- link Cube1: geometry collision box size=1.0344627909428525 1.7002043153528659 0.7150804436725717; visual box size=1.0344627909428525 1.7002043153528659 0.7150804436725717
Joints:
- joint Cube0_Cube1: origin xyz=0.0 0.9276106727308884 1.3566128475401336 rpy=0 0 0 -> xyz=0.14170030557923213 0.0 0.8936453757849808 rpy=0 0 0

Commit message: added code to add sensors in random locations

File: body.urdf (robot description, URDF)
Before this commit: robot robot, 2 links, 1 joints
Links:
- added link Cube2, mass 1; collision box size=1.617463403206064 1.5547374738832658 0.5727068290842984; visual box size=1.617463403206064 1.5547374738832658 0.5727068290842984
- added link Cube3, mass 1; collision box size=0.5022406376745682 0.7017458434279449 1.852951007668724; visual box size=0.5022406376745682 0.7017458434279449 1.852951007668724
- link Cube0: geometry collision box size=1.0835869065506518 1.1751730072125375 0.989398865967424; visual box size=1.0835869065506518 1.1751730072125375 0.989398865967424
- link Cube1: geometry collision box size=1.5511355087122116 1.661030343072863 0.9459327935191741; visual box size=1.5511355087122116 1.661030343072863 0.9459327935191741
Joints:
- added joint Cube1_Cube2: type revolute, parent Cube1, child Cube2, origin xyz=0.7755677543561058 0.0 0.0 rpy=0 0 0, axis 0 1 0, limit lower=-3.14159 upper=3.14159 effort=0.0 velocity=0.0
- added joint Cube2_Cube3: type revolute, parent Cube2, child Cube3, origin xyz=0.808731701603032 0.0 0.0 rpy=0 0 0, axis 0 1 0, limit lower=-3.14159 upper=3.14159 effort=0.0 velocity=0.0
- joint Cube0_Cube1: origin xyz=0.14170030557923213 0.0 0.8936453757849808 rpy=0 0 0 -> xyz=0.27089672663766295 0.0 0.494699432983712 rpy=0 0 0
