Commit message: still struggling with joint placement

File: body.urdf (robot description, URDF)
Before this commit: robot robot, 4 links, 3 joints
Links:
- removed link Cube3
- link Cube0: geometry collision box size=1.659040563610926 1.883305715427261 1.99635995212623; visual box size=1.659040563610926 1.883305715427261 1.99635995212623
- link Cube1: geometry collision box size=1.2230593862469172 0.6549384246153807 1.8864423927541514; visual box size=1.2230593862469172 0.6549384246153807 1.8864423927541514
- link Cube2: geometry collision box size=0.7977519599654331 1.6636483873011678 1.36101370004493; visual box size=0.7977519599654331 1.6636483873011678 1.36101370004493
Joints:
- removed joint Cube2_Cube3
- joint Cube0_Cube1: origin xyz=0.27089672663766295 0.0 0.494699432983712 rpy=0 0 0 -> xyz=0.4147601409027315 0.0 0.998179976063115 rpy=0 0 0
- joint Cube1_Cube2: origin xyz=0.7755677543561058 0.0 0.0 rpy=0 0 0 -> xyz=0.6115296931234586 0.0 0.9432211963770757 rpy=0 0 0

Commit message: links can be different colors

File: body.urdf (robot description, URDF)
Before this commit: robot robot, 3 links, 2 joints
Links:
- added link Cube3, mass 1; collision box size=1.8628996386328915 0.8448482694261172 1.8225398664243722; visual box size=1.8628996386328915 0.8448482694261172 1.8225398664243722
- added link Cube4, mass 1; collision box size=1.4786249326636507 1.5597451112728367 1.7872977242756267; visual box size=1.4786249326636507 1.5597451112728367 1.7872977242756267
- added link Cube5, mass 1; collision box size=1.0313010066961819 0.7778219366049649 1.7418589696845945; visual box size=1.0313010066961819 0.7778219366049649 1.7418589696845945
- added link Cube6, mass 1; collision box size=0.753913427082327 1.4388177394327961 1.774801076261124; visual box size=0.753913427082327 1.4388177394327961 1.774801076261124
- added link Cube7, mass 1; collision box size=1.7693434067666243 0.8551841468130267 1.446227360805167; visual box size=1.7693434067666243 0.8551841468130267 1.446227360805167
- link Cube0: geometry collision box size=1.089836412255409 0.5810732807501715 1.110042479458575; visual box size=1.089836412255409 0.5810732807501715 1.110042479458575
- link Cube1: geometry collision box size=0.9697990063260368 1.2383598515510073 1.2648977762543838; visual box size=0.9697990063260368 1.2383598515510073 1.2648977762543838
- link Cube2: geometry collision box size=1.5435994788279004 0.996516368328823 1.743018573231621; visual box size=1.5435994788279004 0.996516368328823 1.743018573231621
Joints:
- added joint Cube2_Cube3: type revolute, parent Cube2, child Cube3, origin xyz=0.7717997394139502 0.0 0.8715092866158105 rpy=0 0 0, axis 0 1 0, limit lower=-3.14159 upper=3.14159 effort=0.0 velocity=0.0
- added joint Cube3_Cube4: type revolute, parent Cube3, child Cube4, origin xyz=0.9314498193164458 0.0 0.9112699332121861 rpy=0 0 0, axis 0 1 0, limit lower=-3.14159 upper=3.14159 effort=0.0 velocity=0.0
- added joint Cube4_Cube5: type revolute, parent Cube4, child Cube5, origin xyz=0.7393124663318253 0.0 0.8936488621378134 rpy=0 0 0, axis 0 1 0, limit lower=-3.14159 upper=3.14159 effort=0.0 velocity=0.0
- added joint Cube5_Cube6: type revolute, parent Cube5, child Cube6, origin xyz=0.5156505033480909 0.0 0.8709294848422973 rpy=0 0 0, axis 0 1 0, limit lower=-3.14159 upper=3.14159 effort=0.0 velocity=0.0
- added joint Cube6_Cube7: type revolute, parent Cube6, child Cube7, origin xyz=0.3769567135411635 0.0 0.887400538130562 rpy=0 0 0, axis 0 1 0, limit lower=-3.14159 upper=3.14159 effort=0.0 velocity=0.0
- joint Cube0_Cube1: origin xyz=0.4147601409027315 0.0 0.998179976063115 rpy=0 0 0 -> xyz=0.27245910306385224 0.0 0.5550212397292875 rpy=0 0 0
- joint Cube1_Cube2: origin xyz=0.6115296931234586 0.0 0.9432211963770757 rpy=0 0 0 -> xyz=0.4848995031630184 0.0 0.6324488881271919 rpy=0 0 0

Commit message: random joints motorized

File: body.urdf (robot description, URDF)
Before this commit: robot robot, 8 links, 7 joints
Links:
- removed link Cube2
- removed link Cube3
- removed link Cube4
- removed link Cube5
- removed link Cube6
- removed link Cube7
- link Cube0: geometry collision box size=1.3104970524928239 0.8069200459879149 1.0013301985950374; visual box size=1.3104970524928239 0.8069200459879149 1.0013301985950374
- link Cube1: geometry collision box size=0.5681700625671118 1.688915554915399 1.992641160912341; visual box size=0.5681700625671118 1.688915554915399 1.992641160912341
Joints:
- removed joint Cube1_Cube2
- removed joint Cube2_Cube3
- removed joint Cube3_Cube4
- removed joint Cube4_Cube5
- removed joint Cube5_Cube6
- removed joint Cube6_Cube7
- joint Cube0_Cube1: origin xyz=0.27245910306385224 0.0 0.5550212397292875 rpy=0 0 0 -> xyz=0.32762426312320597 0.0 0.5006650992975187 rpy=0 0 0

Commit message: random motors and sensors and synapses between all

File: body.urdf (robot description, URDF)
Before this commit: robot robot, 2 links, 1 joints
Links:
- added link Cube2, mass 1; collision box size=0.2205245017026685 0.6105413304251394 0.7685526998780972; visual box size=0.2205245017026685 0.6105413304251394 0.7685526998780972
- added link Cube3, mass 1; collision box size=0.9744257774128693 1.3327790679724334 0.36221691924218447; visual box size=0.9744257774128693 1.3327790679724334 0.36221691924218447
- added link Cube4, mass 1; collision box size=1.1249213943116942 1.0003427339314683 1.4653957942469666; visual box size=1.1249213943116942 1.0003427339314683 1.4653957942469666
- added link Cube5, mass 1; collision box size=1.0607292957997734 0.5251404192899074 0.2184016551827268; visual box size=1.0607292957997734 0.5251404192899074 0.2184016551827268
- added link Cube6, mass 1; collision box size=1.3200537628211984 0.8045383431858057 0.38505367828217585; visual box size=1.3200537628211984 0.8045383431858057 0.38505367828217585
- link Cube0: geometry collision box size=0.46246486301151224 1.3617453981678458 0.8571598198529593; visual box size=0.46246486301151224 1.3617453981678458 0.8571598198529593
- link Cube1: geometry collision box size=1.475993043931585 0.8116661443237474 0.4820237752274309; visual box size=1.475993043931585 0.8116661443237474 0.4820237752274309
Joints:
- added joint Cube1_Cube2: type revolute, parent Cube1, child Cube2, origin xyz=0.7379965219657925 0.0 0.24101188761371545 rpy=0 0 0, axis 0 1 0, limit lower=-3.14159 upper=3.14159 effort=0.0 velocity=0.0
- added joint Cube2_Cube3: type revolute, parent Cube2, child Cube3, origin xyz=0.11026225085133425 0.0 0.3842763499390486 rpy=0 0 0, axis 0 1 0, limit lower=-3.14159 upper=3.14159 effort=0.0 velocity=0.0
- added joint Cube3_Cube4: type revolute, parent Cube3, child Cube4, origin xyz=0.48721288870643464 0.0 0.18110845962109223 rpy=0 0 0, axis 0 1 0, limit lower=-3.14159 upper=3.14159 effort=0.0 velocity=0.0
- added joint Cube4_Cube5: type revolute, parent Cube4, child Cube5, origin xyz=0.5624606971558471 0.0 0.7326978971234833 rpy=0 0 0, axis 0 1 0, limit lower=-3.14159 upper=3.14159 effort=0.0 velocity=0.0
- added joint Cube5_Cube6: type revolute, parent Cube5, child Cube6, origin xyz=0.5303646478998867 0.0 0.1092008275913634 rpy=0 0 0, axis 0 1 0, limit lower=-3.14159 upper=3.14159 effort=0.0 velocity=0.0
- joint Cube0_Cube1: origin xyz=0.32762426312320597 0.0 0.5006650992975187 rpy=0 0 0 -> xyz=0.11561621575287806 0.0 0.42857990992647965 rpy=0 0 0

Commit message: motorized elements, trying to fix joints

File: body.urdf (robot description, URDF)
Before this commit: robot robot, 7 links, 6 joints
Links:
- removed link Cube3
- removed link Cube4
- removed link Cube5
- removed link Cube6
- link Cube0: geometry collision box size=0.6556339510137397 1.2214824595902019 0.6979547537687409; visual box size=0.6556339510137397 1.2214824595902019 0.6979547537687409
- link Cube1: geometry collision box size=0.9006079054341227 0.6679298401511256 0.6475465952521784; visual box size=0.9006079054341227 0.6679298401511256 0.6475465952521784
- link Cube2: geometry collision box size=1.1403251735334026 0.3038840001813168 1.460559830835901; visual box size=1.1403251735334026 0.3038840001813168 1.460559830835901
Joints:
- removed joint Cube2_Cube3
- removed joint Cube3_Cube4
- removed joint Cube4_Cube5
- removed joint Cube5_Cube6
- joint Cube0_Cube1: origin xyz=0.11561621575287806 0.0 0.42857990992647965 rpy=0 0 0 -> xyz=0.16390848775343492 0.0 0.34897737688437047 rpy=0 0 0
- joint Cube1_Cube2: origin xyz=0.7379965219657925 0.0 0.24101188761371545 rpy=0 0 0 -> xyz=0.45030395271706136 0.0 0.3237732976260892 rpy=0 0 0

Commit message: getting video

File: body.urdf (robot description, URDF)
Before this commit: robot robot, 3 links, 2 joints
Links:
- added link Cube3, mass 1; collision box size=1.2634080986656089 0.5789021242318482 0.3002817285227187; visual box size=1.2634080986656089 0.5789021242318482 0.3002817285227187
- added link Cube4, mass 1; collision box size=0.7040505668630606 0.8886560102843148 0.6056393942324212; visual box size=0.7040505668630606 0.8886560102843148 0.6056393942324212
- added link Cube5, mass 1; collision box size=0.9743193704271249 0.9247997269898502 0.9881569896785134; visual box size=0.9743193704271249 0.9247997269898502 0.9881569896785134
- added link Cube6, mass 1; collision box size=1.3714593871636294 0.5946467689265792 0.39385493973785446; visual box size=1.3714593871636294 0.5946467689265792 0.39385493973785446
- added link Cube7, mass 1; collision box size=0.5714911482073555 0.22598907536395818 1.4993655046047776; visual box size=0.5714911482073555 0.22598907536395818 1.4993655046047776
- added link Cube8, mass 1; collision box size=0.6714161697594784 0.35248737066952096 1.1313702748831118; visual box size=0.6714161697594784 0.35248737066952096 1.1313702748831118
- link Cube0: geometry collision box size=0.9393347805996992 1.342275673665869 0.40847201339990735; visual box size=0.9393347805996992 1.342275673665869 0.40847201339990735
- link Cube1: geometry collision box size=0.5142174661938326 1.4871482072083695 0.27788125430750027; visual box size=0.5142174661938326 1.4871482072083695 0.27788125430750027
- link Cube2: geometry collision box size=0.8973537506117606 1.2816645209818895 1.1367030820750985; visual box size=0.8973537506117606 1.2816645209818895 1.1367030820750985
Joints:
- added joint Cube2_Cube3: type revolute, parent Cube2, child Cube3, origin xyz=0.8973537506117606 0.0 0.0 rpy=0 0 0, axis 0 1 0, limit lower=-3.14159 upper=3.14159 effort=0.0 velocity=0.0
- added joint Cube3_Cube4: type revolute, parent Cube3, child Cube4, origin xyz=1.2634080986656089 0.0 0.0 rpy=0 0 0, axis 0 1 0, limit lower=-3.14159 upper=3.14159 effort=0.0 velocity=0.0
- added joint Cube4_Cube5: type revolute, parent Cube4, child Cube5, origin xyz=0.7040505668630606 0.0 0.0 rpy=0 0 0, axis 0 1 0, limit lower=-3.14159 upper=3.14159 effort=0.0 velocity=0.0
- added joint Cube5_Cube6: type revolute, parent Cube5, child Cube6, origin xyz=0.9743193704271249 0.0 0.0 rpy=0 0 0, axis 0 1 0, limit lower=-3.14159 upper=3.14159 effort=0.0 velocity=0.0
- added joint Cube6_Cube7: type revolute, parent Cube6, child Cube7, origin xyz=1.3714593871636294 0.0 0.0 rpy=0 0 0, axis 0 1 0, limit lower=-3.14159 upper=3.14159 effort=0.0 velocity=0.0
- added joint Cube7_Cube8: type revolute, parent Cube7, child Cube8, origin xyz=0.5714911482073555 0.0 0.0 rpy=0 0 0, axis 0 1 0, limit lower=-3.14159 upper=3.14159 effort=0.0 velocity=0.0
- joint Cube0_Cube1: origin xyz=0.16390848775343492 0.0 0.34897737688437047 rpy=0 0 0 -> xyz=0.4696673902998496 0.0 0.40847201339990735 rpy=0 0 0
- joint Cube1_Cube2: origin xyz=0.45030395271706136 0.0 0.3237732976260892 rpy=0 0 0 -> xyz=0.5142174661938326 0.0 0.0 rpy=0 0 0

Commit message: added videos

File: body.urdf (robot description, URDF)
Before this commit: robot robot, 9 links, 8 joints
Links:
- added link Cube9, mass 1; collision box size=0.8784294836398616 0.7264944207367168 0.9169304662787383; visual box size=0.8784294836398616 0.7264944207367168 0.9169304662787383
- link Cube0: geometry collision box size=1.4162648333887855 0.5958564672642277 1.1737275009717258; visual box size=1.4162648333887855 0.5958564672642277 1.1737275009717258
- link Cube1: geometry collision box size=0.5542559880171682 1.3719595992065137 0.6151404245278305; visual box size=0.5542559880171682 1.3719595992065137 0.6151404245278305
- link Cube2: geometry collision box size=0.7793290827231101 1.1862708498460999 1.1684708418728338; visual box size=0.7793290827231101 1.1862708498460999 1.1684708418728338
- link Cube3: geometry collision box size=0.7014656026491273 0.9244912166348469 0.8650249255165048; visual box size=0.7014656026491273 0.9244912166348469 0.8650249255165048
- link Cube4: geometry collision box size=1.467682328368379 0.7020664417060909 0.41955477065732194; visual box size=1.467682328368379 0.7020664417060909 0.41955477065732194
- link Cube5: geometry collision box size=1.2252069638311842 0.6931602885638961 1.419943749625771; visual box size=1.2252069638311842 0.6931602885638961 1.419943749625771
- link Cube6: geometry collision box size=0.4836830933446293 1.2922839138159177 0.8825199189658672; visual box size=0.4836830933446293 1.2922839138159177 0.8825199189658672
- link Cube7: geometry collision box size=0.9363832848796578 0.9917380207871453 0.7497096486046053; visual box size=0.9363832848796578 0.9917380207871453 0.7497096486046053
- link Cube8: geometry collision box size=1.3192789089283212 0.6996738511611821 0.3557826717563976; visual box size=1.3192789089283212 0.6996738511611821 0.3557826717563976
Joints:
- added joint Cube8_Cube9: type revolute, parent Cube8, child Cube9, origin xyz=1.3192789089283212 0.0 0.0 rpy=0 0 0, axis 0 1 0, limit lower=-3.14159 upper=3.14159 effort=0.0 velocity=0.0
- joint Cube0_Cube1: origin xyz=0.4696673902998496 0.0 0.40847201339990735 rpy=0 0 0 -> xyz=0.7081324166943928 0.0 1.1737275009717258 rpy=0 0 0
- joint Cube1_Cube2: origin xyz=0.5142174661938326 0.0 0.0 rpy=0 0 0 -> xyz=0.5542559880171682 0.0 0.0 rpy=0 0 0
- joint Cube2_Cube3: origin xyz=0.8973537506117606 0.0 0.0 rpy=0 0 0 -> xyz=0.7793290827231101 0.0 0.0 rpy=0 0 0
- joint Cube3_Cube4: origin xyz=1.2634080986656089 0.0 0.0 rpy=0 0 0 -> xyz=0.7014656026491273 0.0 0.0 rpy=0 0 0
- joint Cube4_Cube5: origin xyz=0.7040505668630606 0.0 0.0 rpy=0 0 0 -> xyz=1.467682328368379 0.0 0.0 rpy=0 0 0
- joint Cube5_Cube6: origin xyz=0.9743193704271249 0.0 0.0 rpy=0 0 0 -> xyz=1.2252069638311842 0.0 0.0 rpy=0 0 0
- joint Cube6_Cube7: origin xyz=1.3714593871636294 0.0 0.0 rpy=0 0 0 -> xyz=0.4836830933446293 0.0 0.0 rpy=0 0 0
- joint Cube7_Cube8: origin xyz=0.5714911482073555 0.0 0.0 rpy=0 0 0 -> xyz=0.9363832848796578 0.0 0.0 rpy=0 0 0

Commit message: seems to be working with one bigger loop

File: body.urdf (robot description, URDF)
Before this commit: robot robot, 10 links, 9 joints
Links:
- removed link Cube5
- removed link Cube6
- removed link Cube7
- removed link Cube8
- removed link Cube9
- link Cube0: geometry collision box size=0.4245906286042044 0.4081494047609957 0.5745854030037043; visual box size=0.4245906286042044 0.4081494047609957 0.5745854030037043
- link Cube1: geometry collision box size=0.45222821948713915 1.0971783421744834 0.5773281728999081; visual box size=0.45222821948713915 1.0971783421744834 0.5773281728999081
- link Cube2: geometry collision box size=0.7524666172487486 1.4561803317211874 1.488488966020785; visual box size=0.7524666172487486 1.4561803317211874 1.488488966020785
- link Cube3: geometry collision box size=1.0300319335776638 1.0324790929476233 0.6238794634484706; visual box size=1.0300319335776638 1.0324790929476233 0.6238794634484706
- link Cube4: geometry collision box size=0.8909267229726481 0.7448161818447459 0.6804117718113273; visual box size=0.8909267229726481 0.7448161818447459 0.6804117718113273
Joints:
- removed joint Cube4_Cube5
- removed joint Cube5_Cube6
- removed joint Cube6_Cube7
- removed joint Cube7_Cube8
- removed joint Cube8_Cube9
- joint Cube0_Cube1: origin xyz=0.7081324166943928 0.0 1.1737275009717258 rpy=0 0 0 -> xyz=0.2122953143021022 0.0 0.5745854030037043 rpy=0 0 0
- joint Cube1_Cube2: origin xyz=0.5542559880171682 0.0 0.0 rpy=0 0 0 -> xyz=0.45222821948713915 0.0 0.0 rpy=0 0 0
- joint Cube2_Cube3: origin xyz=0.7793290827231101 0.0 0.0 rpy=0 0 0 -> xyz=0.7524666172487486 0.0 0.0 rpy=0 0 0
- joint Cube3_Cube4: origin xyz=0.7014656026491273 0.0 0.0 rpy=0 0 0 -> xyz=1.0300319335776638 0.0 0.0 rpy=0 0 0

Commit message: adds blocks to the side?

File: body.urdf (robot description, URDF)
Before this commit: robot robot, 5 links, 4 joints
Links:
- removed link Cube3
- removed link Cube4
- link Cube0: geometry collision box size=1.313376433186252 1.402939989935109 1.2569446628047225; visual box size=1.313376433186252 1.402939989935109 1.2569446628047225
- link Cube1: geometry collision box size=0.6012379550952679 0.4920962371999745 1.260898693454427; visual box size=0.6012379550952679 0.4920962371999745 1.260898693454427
- link Cube2: geometry collision box size=0.5534911286327533 0.36404166456978787 0.28071742468799676; visual box size=0.5534911286327533 0.36404166456978787 0.28071742468799676
Joints:
- removed joint Cube2_Cube3
- removed joint Cube3_Cube4
- joint Cube0_Cube1: origin xyz=0.2122953143021022 0.0 0.5745854030037043 rpy=0 0 0 -> xyz=0.0 0.0 1.7430553371952775 rpy=0 0 0
- joint Cube1_Cube2: origin xyz=0.45222821948713915 0.0 0.0 rpy=0 0 0 -> xyz=0.0 0.0 -1.260898693454427 rpy=0 0 0

Commit message: grow well in straight y direction

File: body.urdf (robot description, URDF)
Before this commit: robot robot, 3 links, 2 joints
Links:
- added link Cube3, mass 1; collision box size=0.597892703260761 0.207056178437718 0.3979462418004306; visual box size=0.597892703260761 0.207056178437718 0.3979462418004306
- added link Cube4, mass 1; collision box size=0.424786898700399 0.2341197291400388 0.3899182518469194; visual box size=0.424786898700399 0.2341197291400388 0.3899182518469194
- link Cube0: geometry collision box size=1.3022791340964648 0.2628779242540864 0.40833645292269705; visual box size=1.3022791340964648 0.2628779242540864 0.40833645292269705
- link Cube1: geometry collision box size=0.9742062204343507 0.20106935729348985 0.25002224246465726; visual box size=0.9742062204343507 0.20106935729348985 0.25002224246465726
- link Cube2: geometry collision box size=0.2856398400322672 0.2185459408756211 0.3742690679452231; visual box size=0.2856398400322672 0.2185459408756211 0.3742690679452231
Joints:
- added joint Cube2_Cube3: type revolute, parent Cube2, child Cube3, origin xyz=0.0 -0.2185459408756211 0.0 rpy=0 0 0, axis 0 1 0, limit lower=-3.14159 upper=3.14159 effort=0.0 velocity=0.0
- added joint Cube3_Cube4: type revolute, parent Cube3, child Cube4, origin xyz=0.0 -0.207056178437718 0.0 rpy=0 0 0, axis 0 1 0, limit lower=-3.14159 upper=3.14159 effort=0.0 velocity=0.0
- joint Cube0_Cube1: origin xyz=0.0 0.0 1.7430553371952775 rpy=0 0 0 -> xyz=0.0 -0.1314389621270432 3 rpy=0 0 0
- joint Cube1_Cube2: origin xyz=0.0 0.0 -1.260898693454427 rpy=0 0 0 -> xyz=0.0 -0.20106935729348985 0.0 rpy=0 0 0

Commit message: legs generate correctly, going to the side and down

File: body.urdf (robot description, URDF)
Before this commit: robot robot, 5 links, 4 joints
Links:
- link Cube0: geometry collision box size=0.9521840403561987 0.48785834157389046 0.32373948053526347; visual box size=0.9521840403561987 0.48785834157389046 0.32373948053526347
- link Cube1: geometry collision box size=0.943554041028424 0.40005091664347436 0.2321112295434946; visual box size=0.943554041028424 0.40005091664347436 0.2321112295434946
- link Cube2: geometry collision box size=0.5803995108054099 0.2087690966301285 0.2935161531443098; visual box size=0.5803995108054099 0.2087690966301285 0.2935161531443098
- link Cube3: geometry collision box size=0.2538313697896991 0.43151102470584324 0.26244529633387736; visual box size=0.2538313697896991 0.43151102470584324 0.26244529633387736
- link Cube4: geometry collision box size=0.5333121073175191 0.3879550964967629 0.23079355293584927; visual box size=0.5333121073175191 0.3879550964967629 0.23079355293584927
Joints:
- joint Cube0_Cube1: origin xyz=0.0 -0.1314389621270432 3 rpy=0 0 0 -> xyz=0.0 -0.24392917078694523 3 rpy=0 0 0
- joint Cube1_Cube2: origin xyz=0.0 -0.20106935729348985 0.0 rpy=0 0 0 -> xyz=0.0 -0.20002545832173718 -0.1160556147717473 rpy=0 0 0
- joint Cube2_Cube3: origin xyz=0.0 -0.2185459408756211 0.0 rpy=0 0 0 -> xyz=0.0 0.0 -0.2935161531443098 rpy=0 0 0
- joint Cube3_Cube4: origin xyz=0.0 -0.207056178437718 0.0 rpy=0 0 0 -> xyz=0.0 -0.21575551235292162 -0.13122264816693868 rpy=0 0 0

Commit message: one side with 1 vertebrae link seems to be working well! sensors and motors randomly added as well

File: body.urdf (robot description, URDF)
Before this commit: robot robot, 5 links, 4 joints
Links:
- link Cube0: geometry collision box size=0.2755966989832326 1.4261487098564691 0.7969218791989545; visual box size=0.2755966989832326 1.4261487098564691 0.7969218791989545
- link Cube1: geometry collision box size=0.2590128849418823 1.406967845475562 0.5138442557023681; visual box size=0.2590128849418823 1.406967845475562 0.5138442557023681
- link Cube2: geometry collision box size=0.21324183840988356 0.716985632020426 0.5809221966252599; visual box size=0.21324183840988356 0.716985632020426 0.5809221966252599
- link Cube3: geometry collision box size=0.21845478051937142 0.4185114926964161 0.5524604507985196; visual box size=0.21845478051937142 0.4185114926964161 0.5524604507985196
- link Cube4: geometry collision box size=0.23969804941713796 1.0057856371316607 0.66814938041945; visual box size=0.23969804941713796 1.0057856371316607 0.66814938041945
Joints:
- joint Cube0_Cube1: origin xyz=0.0 -0.24392917078694523 3 rpy=0 0 0 -> xyz=0.0 -0.7130743549282346 3 rpy=0 0 0; type revolute -> prismatic
- joint Cube1_Cube2: origin xyz=0.0 -0.20002545832173718 -0.1160556147717473 rpy=0 0 0 -> xyz=0.0 -0.703483922737781 -0.25692212785118407 rpy=0 0 0; type revolute -> prismatic
- joint Cube2_Cube3: origin xyz=0.0 0.0 -0.2935161531443098 rpy=0 0 0 -> xyz=0.0 0.0 -0.5809221966252599 rpy=0 0 0; type revolute -> fixed
- joint Cube3_Cube4: origin xyz=0.0 -0.21575551235292162 -0.13122264816693868 rpy=0 0 0 -> xyz=0.0 -0.20925574634820804 -0.2762302253992598 rpy=0 0 0
