Commit message: builds legs on either side of a vertebrae using a loop

File: body.urdf (robot description, URDF)
Before this commit: robot robot, 5 links, 4 joints
Links:
- added link Cube5, mass 1; collision box size=0.6417191004565326 0.23448640764110348 0.2579857603423419; visual box size=0.6417191004565326 0.23448640764110348 0.2579857603423419
- added link Cube6, mass 1; collision box size=0.7407438708422376 0.2206232862167036 0.20557429029422739; visual box size=0.7407438708422376 0.2206232862167036 0.20557429029422739
- added link Cube7, mass 1; collision box size=0.9637879053241933 0.25050106875575723 0.2991036579670061; visual box size=0.9637879053241933 0.25050106875575723 0.2991036579670061
- added link Cube8, mass 1; collision box size=0.6936367946728837 0.20042818523441955 0.22758302614990142; visual box size=0.6936367946728837 0.20042818523441955 0.22758302614990142
- link Cube0: geometry collision box size=1.1459338181466834 0.2762827722053154 0.32238620168864496; visual box size=1.1459338181466834 0.2762827722053154 0.32238620168864496
- link Cube1: geometry collision box size=0.28533981183273444 0.26329359395871393 0.28656500589533096; visual box size=0.28533981183273444 0.26329359395871393 0.28656500589533096
- link Cube2: geometry collision box size=0.6784111604526679 0.2666296738798568 0.2377897537539046; visual box size=0.6784111604526679 0.2666296738798568 0.2377897537539046
- link Cube3: geometry collision box size=0.3089585581996639 0.2523203994933851 0.29003245192973215; visual box size=0.3089585581996639 0.2523203994933851 0.29003245192973215
- link Cube4: geometry collision box size=0.9146439731715064 0.2745234242995004 0.2476366217627384; visual box size=0.9146439731715064 0.2745234242995004 0.2476366217627384
Joints:
- added joint Cube0_Cube5: type spherical, parent Cube0, child Cube5, origin xyz=0.0 0.1381413861026577 3 rpy=0 0 0, axis 0 1 0, limit lower=-3.14159 upper=3.14159 effort=0.0 velocity=0.0
- added joint Cube5_Cube6: type prismatic, parent Cube5, child Cube6, origin xyz=0.0 0.11724320382055174 -0.12899288017117094 rpy=0 0 0, axis 0 1 0, limit lower=-3.14159 upper=3.14159 effort=0.0 velocity=0.0
- added joint Cube6_Cube7: type fixed, parent Cube6, child Cube7, origin xyz=0.0 0.0 -0.20557429029422739 rpy=0 0 0, axis 0 1 0, limit lower=-3.14159 upper=3.14159 effort=0.0 velocity=0.0
- added joint Cube7_Cube8: type fixed, parent Cube7, child Cube8, origin xyz=0.0 0.12525053437787861 -0.14955182898350305 rpy=0 0 0, axis 0 1 0, limit lower=-3.14159 upper=3.14159 effort=0.0 velocity=0.0
- joint Cube0_Cube1: origin xyz=0.0 -0.7130743549282346 3 rpy=0 0 0 -> xyz=0.0 -0.1381413861026577 3 rpy=0 0 0; type prismatic -> fixed
- joint Cube1_Cube2: origin xyz=0.0 -0.703483922737781 -0.25692212785118407 rpy=0 0 0 -> xyz=0.0 -0.26329359395871393 0.0 rpy=0 0 0
- joint Cube2_Cube3: origin xyz=0.0 0.0 -0.5809221966252599 rpy=0 0 0 -> xyz=0.0 -0.2666296738798568 0.0 rpy=0 0 0; type fixed -> revolute
- joint Cube3_Cube4: origin xyz=0.0 -0.20925574634820804 -0.2762302253992598 rpy=0 0 0 -> xyz=0.0 -0.12616019974669254 -0.14501622596486607 rpy=0 0 0

Commit message: generates random of 1 vertebrae with each cube decreasing in size, now trying to extend

File: body.urdf (robot description, URDF)
Before this commit: robot robot, 9 links, 8 joints
Links:
- link Cube0: geometry collision box size=0.8145772649644409 0.4519505274883279 1.1980158883149175; visual box size=0.8145772649644409 0.4519505274883279 1.1980158883149175
- link Cube1: geometry collision box size=0.2714750409511145 0.4207837629736487 0.36833436123921337; visual box size=0.2714750409511145 0.4207837629736487 0.36833436123921337
- link Cube2: geometry collision box size=0.23995323279351577 0.4029792531627467 0.34195311549170115; visual box size=0.23995323279351577 0.4029792531627467 0.34195311549170115
- link Cube3: geometry collision box size=0.22567648459172476 0.363633235994984 0.20743170699853433; visual box size=0.22567648459172476 0.363633235994984 0.20743170699853433
- link Cube4: geometry collision box size=0.21658726463792372 0.22442932471869081 0.20531546685474641; visual box size=0.21658726463792372 0.22442932471869081 0.20531546685474641
- link Cube5: geometry collision box size=0.2043417133497992 0.21607272838430353 0.20003031601087348; visual box size=0.2043417133497992 0.21607272838430353 0.20003031601087348
- link Cube6: geometry collision box size=0.20331148857830972 0.21336843035117808 0.20000343036677945; visual box size=0.20331148857830972 0.21336843035117808 0.20000343036677945
- link Cube7: geometry collision box size=0.20204503580774427 0.2128688729867195 0.20000126410251187; visual box size=0.20204503580774427 0.2128688729867195 0.20000126410251187
- link Cube8: geometry collision box size=0.20200871991388877 0.2029158914420766 0.20000016176146881; visual box size=0.20200871991388877 0.2029158914420766 0.20000016176146881
Joints:
- joint Cube0_Cube1: origin xyz=0.0 -0.1381413861026577 3 rpy=0 0 0 -> xyz=0.0 -0.22597526374416396 3 rpy=0 0 0; type fixed -> revolute
- joint Cube0_Cube5: origin xyz=0.0 0.1381413861026577 3 rpy=0 0 0 -> xyz=0.0 0.22597526374416396 3 rpy=0 0 0
- joint Cube1_Cube2: origin xyz=0.0 -0.26329359395871393 0.0 rpy=0 0 0 -> xyz=0.0 -0.21039188148682436 -0.18416718061960669 rpy=0 0 0; type prismatic -> fixed
- joint Cube2_Cube3: origin xyz=0.0 -0.2666296738798568 0.0 rpy=0 0 0 -> xyz=0.0 0.0 -0.34195311549170115 rpy=0 0 0; type revolute -> spherical
- joint Cube3_Cube4: origin xyz=0.0 -0.12616019974669254 -0.14501622596486607 rpy=0 0 0 -> xyz=0.0 0.0 -0.20743170699853433 rpy=0 0 0; type revolute -> fixed
- joint Cube5_Cube6: origin xyz=0.0 0.11724320382055174 -0.12899288017117094 rpy=0 0 0 -> xyz=0.0 0.10803636419215176 -0.10001515800543674 rpy=0 0 0; type prismatic -> revolute
- joint Cube6_Cube7: origin xyz=0.0 0.0 -0.20557429029422739 rpy=0 0 0 -> xyz=0.0 0.10668421517558904 -0.10000171518338972 rpy=0 0 0
- joint Cube7_Cube8: origin xyz=0.0 0.12525053437787861 -0.14955182898350305 rpy=0 0 0 -> xyz=0.0 0.10643443649335975 -0.10000063205125594 rpy=0 0 0; type fixed -> prismatic

Commit message: can add one vertebrae link no legs

File: body.urdf (robot description, URDF)
Before this commit: robot robot, 9 links, 8 joints
Links:
- added link Cube10, mass 1; collision box size=0.20000890787928652 0.20000331749394482 0.2002191770413995; visual box size=0.20000890787928652 0.20000331749394482 0.2002191770413995
- added link Cube11, mass 1; collision box size=1.0130812819027917 1.1482431570090235 0.4762095113668587; visual box size=1.0130812819027917 1.1482431570090235 0.4762095113668587
- added link Cube9, mass 1; collision box size=0.20001428362684998 0.20000564399569404 0.2003452596367829; visual box size=0.20001428362684998 0.20000564399569404 0.2003452596367829
- link Cube0: geometry collision box size=1.380748693585828 0.5695275888188964 1.3964472608721477; visual box size=1.380748693585828 0.5695275888188964 1.3964472608721477
- link Cube1: geometry collision box size=0.2354094027108493 0.32514961074209503 0.5645914776251995; visual box size=0.2354094027108493 0.32514961074209503 0.5645914776251995
- link Cube2: geometry collision box size=0.2088563580229962 0.2764143365151802 0.27847965885466813; visual box size=0.2088563580229962 0.2764143365151802 0.27847965885466813
- link Cube3: geometry collision box size=0.207941660181239 0.2034441321977377 0.24686363105354864; visual box size=0.207941660181239 0.2034441321977377 0.24686363105354864
- link Cube4: geometry collision box size=0.2018793434731679 0.2007477443702796 0.2288526377215384; visual box size=0.2018793434731679 0.2007477443702796 0.2288526377215384
- link Cube5: geometry collision box size=0.20131472150375854 0.2007325026821564 0.21503682136069457; visual box size=0.20131472150375854 0.2007325026821564 0.21503682136069457
- link Cube6: geometry collision box size=0.20076301136736557 0.20040536503272716 0.21114819401667975; visual box size=0.20076301136736557 0.20040536503272716 0.21114819401667975
- link Cube7: geometry collision box size=0.2001374430350857 0.20003249251663685 0.20256528226116557; visual box size=0.2001374430350857 0.20003249251663685 0.20256528226116557
- link Cube8: geometry collision box size=0.20001753150432475 0.20001216182368703 0.20243866216696285; visual box size=0.20001753150432475 0.20001216182368703 0.20243866216696285
Joints:
- removed joint Cube0_Cube5
- removed joint Cube5_Cube6
- added joint Cube0_Cube11: type revolute, parent Cube0, child Cube11, origin xyz=0.690374346792914 0.0 3 rpy=0 0 0, axis 0 1 0, limit lower=-3.14159 upper=3.14159 effort=0.0 velocity=0.0
- added joint Cube0_Cube6: type spherical, parent Cube0, child Cube6, origin xyz=0.0 0.2847637944094482 3 rpy=0 0 0, axis 0 1 0, limit lower=-3.14159 upper=3.14159 effort=0.0 velocity=0.0
- added joint Cube4_Cube5: type fixed, parent Cube4, child Cube5, origin xyz=0.0 -0.1003738721851398 -0.1144263188607692 rpy=0 0 0, axis 0 1 0, limit lower=-3.14159 upper=3.14159 effort=0.0 velocity=0.0
- added joint Cube8_Cube9: type prismatic, parent Cube8, child Cube9, origin xyz=0.0 0.0 -0.20243866216696285 rpy=0 0 0, axis 0 1 0, limit lower=-3.14159 upper=3.14159 effort=0.0 velocity=0.0
- added joint Cube9_Cube10: type spherical, parent Cube9, child Cube10, origin xyz=0.0 0.10000282199784702 -0.10017262981839145 rpy=0 0 0, axis 0 1 0, limit lower=-3.14159 upper=3.14159 effort=0.0 velocity=0.0
- joint Cube0_Cube1: origin xyz=0.0 -0.22597526374416396 3 rpy=0 0 0 -> xyz=0.0 -0.2847637944094482 3 rpy=0 0 0; type revolute -> prismatic
- joint Cube1_Cube2: origin xyz=0.0 -0.21039188148682436 -0.18416718061960669 rpy=0 0 0 -> xyz=0.0 -0.16257480537104751 -0.28229573881259973 rpy=0 0 0; type fixed -> prismatic
- joint Cube2_Cube3: origin xyz=0.0 0.0 -0.34195311549170115 rpy=0 0 0 -> xyz=0.0 0.0 -0.27847965885466813 rpy=0 0 0; type spherical -> revolute
- joint Cube3_Cube4: origin xyz=0.0 0.0 -0.20743170699853433 rpy=0 0 0 -> xyz=0.0 -0.10172206609886884 -0.12343181552677432 rpy=0 0 0
- joint Cube6_Cube7: origin xyz=0.0 0.10668421517558904 -0.10000171518338972 rpy=0 0 0 -> xyz=0.0 0.10020268251636358 -0.10557409700833988 rpy=0 0 0; type fixed -> spherical
- joint Cube7_Cube8: origin xyz=0.0 0.10643443649335975 -0.10000063205125594 rpy=0 0 0 -> xyz=0.0 0.0 -0.20256528226116557 rpy=0 0 0

Commit message: correct height of extra legs but incorrect starting point in y

File: body.urdf (robot description, URDF)
Before this commit: robot robot, 12 links, 11 joints
Links:
- added link Cube12, mass 1; collision box size=0.2148293737181759 0.20120528028139614 0.20048658990888657; visual box size=0.2148293737181759 0.20120528028139614 0.20048658990888657
- added link Cube13, mass 1; collision box size=0.2529392106142521 0.6130545861256949 0.48451346340998924; visual box size=0.2529392106142521 0.6130545861256949 0.48451346340998924
- added link Cube14, mass 1; collision box size=0.20502393084563325 0.5425051090252601 0.44121413368637064; visual box size=0.20502393084563325 0.5425051090252601 0.44121413368637064
- added link Cube15, mass 1; collision box size=0.20070193544662238 0.2760155107882258 0.42149359291587035; visual box size=0.20070193544662238 0.2760155107882258 0.42149359291587035
- added link Cube16, mass 1; collision box size=0.8170859718645478 0.4580672808912212 1.0321203909133392; visual box size=0.8170859718645478 0.4580672808912212 1.0321203909133392
- link Cube0: geometry collision box size=0.5691551599968232 1.1324055278794294 0.7194174599007652; visual box size=0.5691551599968232 1.1324055278794294 0.7194174599007652
- link Cube1: geometry collision box size=0.5592876305349179 0.4148458006776878 0.3328471412204361; visual box size=0.5592876305349179 0.4148458006776878 0.3328471412204361
- link Cube10: geometry collision box size=0.2647208960757257 0.2052760662150136 0.20144470236899767; visual box size=0.2647208960757257 0.2052760662150136 0.20144470236899767
- link Cube11: geometry collision box size=0.21839400217827268 0.20127807042695575 0.20079505147913354; visual box size=0.21839400217827268 0.20127807042695575 0.20079505147913354
- link Cube2: geometry collision box size=0.29818790635638837 0.3283339273637037 0.2455740320331536; visual box size=0.29818790635638837 0.3283339273637037 0.2455740320331536
- link Cube3: geometry collision box size=0.266909969185784 0.2492338121604057 0.22814025852025574; visual box size=0.266909969185784 0.2492338121604057 0.22814025852025574
- link Cube4: geometry collision box size=0.21706255661865037 0.20426890607994547 0.21127775047554995; visual box size=0.21706255661865037 0.20426890607994547 0.21127775047554995
- link Cube5: geometry collision box size=0.846528374948339 0.9622221546895064 1.257013683987033; visual box size=0.846528374948339 0.9622221546895064 1.257013683987033
- link Cube6: geometry collision box size=0.7892015128150536 0.5068184669513904 0.6534733584202013; visual box size=0.7892015128150536 0.5068184669513904 0.6534733584202013
- link Cube7: geometry collision box size=0.6200145591017643 0.46343862101893635 0.3715246451011497; visual box size=0.6200145591017643 0.46343862101893635 0.3715246451011497
- link Cube8: geometry collision box size=0.4810780159069635 0.33376171808682265 0.2240533936933442; visual box size=0.4810780159069635 0.33376171808682265 0.2240533936933442
- link Cube9: geometry collision box size=0.32892726883721163 0.20915522185902638 0.2119688440904635; visual box size=0.32892726883721163 0.20915522185902638 0.2119688440904635
Joints:
- removed joint Cube0_Cube11
- removed joint Cube0_Cube6
- removed joint Cube3_Cube4
- removed joint Cube4_Cube5
- removed joint Cube8_Cube9
- added joint Cube0_Cube4: type revolute, parent Cube0, child Cube4, origin xyz=0.0 0.5662027639397147 3 rpy=0 0 0, axis 0 1 0, limit lower=-3.14159 upper=3.14159 effort=0.0 velocity=0.0
- added joint Cube0_Cube5: type revolute, parent Cube0, child Cube5, origin xyz=0.2845775799984116 0.0 3 rpy=0 0 0, axis 0 1 0, limit lower=-3.14159 upper=3.14159 effort=0.0 velocity=0.0
- added joint Cube10_Cube11: type revolute, parent Cube10, child Cube11, origin xyz=0.0 0.1026380331075068 -0.10072235118449883 rpy=0 0 0, axis 0 1 0, limit lower=-3.14159 upper=3.14159 effort=0.0 velocity=0.0
- added joint Cube11_Cube12: type revolute, parent Cube11, child Cube12, origin xyz=0.0 0.0 -0.20079505147913354 rpy=0 0 0, axis 0 1 0, limit lower=-3.14159 upper=3.14159 effort=0.0 velocity=0.0
- added joint Cube13_Cube14: type revolute, parent Cube13, child Cube14, origin xyz=0.0 -0.30652729306284743 0.0 rpy=0 0 0, axis 0 1 0, limit lower=-3.14159 upper=3.14159 effort=0.0 velocity=0.0
- added joint Cube13_Cube16: type revolute, parent Cube13, child Cube16, origin xyz=0.2529392106142521 0.0 0.0 rpy=0 0 0, axis 0 1 0, limit lower=-3.14159 upper=3.14159 effort=0.0 velocity=0.0
- added joint Cube14_Cube15: type revolute, parent Cube14, child Cube15, origin xyz=0.0 -0.27125255451263003 -0.22060706684318532 rpy=0 0 0, axis 0 1 0, limit lower=-3.14159 upper=3.14159 effort=0.0 velocity=0.0
- added joint Cube5_Cube13: type revolute, parent Cube5, child Cube13, origin xyz=0.846528374948339 0.0 0.0 rpy=0 0 0, axis 0 1 0, limit lower=-3.14159 upper=3.14159 effort=0.0 velocity=0.0
- added joint Cube5_Cube6: type revolute, parent Cube5, child Cube6, origin xyz=0.0 -0.4811110773447532 0.0 rpy=0 0 0, axis 0 1 0, limit lower=-3.14159 upper=3.14159 effort=0.0 velocity=0.0
- added joint Cube5_Cube9: type revolute, parent Cube5, child Cube9, origin xyz=0.0 0.4811110773447532 0.0 rpy=0 0 0, axis 0 1 0, limit lower=-3.14159 upper=3.14159 effort=0.0 velocity=0.0
- joint Cube0_Cube1: origin xyz=0.0 -0.2847637944094482 3 rpy=0 0 0 -> xyz=0.0 -0.5662027639397147 3 rpy=0 0 0; type prismatic -> revolute
- joint Cube1_Cube2: origin xyz=0.0 -0.16257480537104751 -0.28229573881259973 rpy=0 0 0 -> xyz=0.0 -0.2074229003388439 -0.16642357061021806 rpy=0 0 0; type prismatic -> revolute
- joint Cube2_Cube3: origin xyz=0.0 0.0 -0.27847965885466813 rpy=0 0 0 -> xyz=0.0 0.0 -0.2455740320331536 rpy=0 0 0
- joint Cube6_Cube7: origin xyz=0.0 0.10020268251636358 -0.10557409700833988 rpy=0 0 0 -> xyz=0.0 -0.2534092334756952 -0.32673667921010063 rpy=0 0 0; type spherical -> revolute
- joint Cube7_Cube8: origin xyz=0.0 0.0 -0.20256528226116557 rpy=0 0 0 -> xyz=0.0 -0.23171931050946817 -0.18576232255057484 rpy=0 0 0; type prismatic -> revolute
- joint Cube9_Cube10: origin xyz=0.0 0.10000282199784702 -0.10017262981839145 rpy=0 0 0 -> xyz=0.0 0.20915522185902638 0.0 rpy=0 0 0; type spherical -> revolute

Commit message: working! just gonna get video

File: body.urdf (robot description, URDF)
Before this commit: robot robot, 17 links, 16 joints
Links:
- removed link Cube15
- removed link Cube16
- link Cube0: geometry collision box size=0.3017352493162563 1.1499378881277058 0.8384181315752945; visual box size=0.3017352493162563 1.1499378881277058 0.8384181315752945
- link Cube1: geometry collision box size=0.26811561673452017 0.7880995429068027 0.4182990373218688; visual box size=0.26811561673452017 0.7880995429068027 0.4182990373218688
- link Cube10: geometry collision box size=0.24515534118506274 0.43793028801041534 0.3879571855421595; visual box size=0.24515534118506274 0.43793028801041534 0.3879571855421595
- link Cube11: geometry collision box size=0.21179066739673846 0.39526688903506585 0.35040553551073245; visual box size=0.21179066739673846 0.39526688903506585 0.35040553551073245
- link Cube12: geometry collision box size=0.2007839871495418 0.27015081469609736 0.3026504017346556; visual box size=0.2007839871495418 0.27015081469609736 0.3026504017346556
- link Cube13: geometry collision box size=0.20074829454977056 0.25526976966486653 0.28860604792426525; visual box size=0.20074829454977056 0.25526976966486653 0.28860604792426525
- link Cube14: geometry collision box size=1.3897893774013899 1.2702127336510136 0.814065042075846; visual box size=1.3897893774013899 1.2702127336510136 0.814065042075846
- link Cube2: geometry collision box size=0.2330897974952698 0.35783070520894994 0.3147667609680614; visual box size=0.2330897974952698 0.35783070520894994 0.3147667609680614
- link Cube3: geometry collision box size=0.2071284014535964 0.2045384180145826 0.24951155584882573; visual box size=0.2071284014535964 0.2045384180145826 0.24951155584882573
- link Cube4: geometry collision box size=0.2051391406605549 0.20449618151733956 0.2281474025343521; visual box size=0.2051391406605549 0.20449618151733956 0.2281474025343521
- link Cube5: geometry collision box size=0.2038705112191872 0.20387926084840882 0.22678881682032553; visual box size=0.2038705112191872 0.20387926084840882 0.22678881682032553
- link Cube6: geometry collision box size=0.20257323337283592 0.20064304174729147 0.2027091076707052; visual box size=0.20257323337283592 0.20064304174729147 0.2027091076707052
- link Cube7: geometry collision box size=0.33345319835012854 1.0195205142971724 1.4726612171863405; visual box size=0.33345319835012854 1.0195205142971724 1.4726612171863405
- link Cube8: geometry collision box size=0.31997294635743173 0.6697136961965823 1.0938645006619618; visual box size=0.31997294635743173 0.6697136961965823 1.0938645006619618
- link Cube9: geometry collision box size=0.317743335549183 0.6104663571604139 0.43865901717092065; visual box size=0.317743335549183 0.6104663571604139 0.43865901717092065
Joints:
- removed joint Cube0_Cube4
- removed joint Cube10_Cube11
- removed joint Cube13_Cube14
- removed joint Cube13_Cube16
- removed joint Cube14_Cube15
- removed joint Cube5_Cube13
- removed joint Cube5_Cube9
- removed joint Cube6_Cube7
- added joint Cube0_Cube7: type revolute, parent Cube0, child Cube7, origin xyz=0.15086762465812814 0.0 3 rpy=0 0 0, axis 0 1 0, limit lower=-3.14159 upper=3.14159 effort=0.0 velocity=0.0
- added joint Cube12_Cube13: type revolute, parent Cube12, child Cube13, origin xyz=0.0 0.0 -0.3026504017346556 rpy=0 0 0, axis 0 1 0, limit lower=-3.14159 upper=3.14159 effort=0.0 velocity=0.0
- added joint Cube3_Cube4: type revolute, parent Cube3, child Cube4, origin xyz=0.0 -0.1022692090072913 -0.12475577792441286 rpy=0 0 0, axis 0 1 0, limit lower=-3.14159 upper=3.14159 effort=0.0 velocity=0.0
- added joint Cube7_Cube11: type revolute, parent Cube7, child Cube11, origin xyz=-0.16672659917506427 0.5097602571485862 0.0 rpy=0 0 0, axis 0 1 0, limit lower=-3.14159 upper=3.14159 effort=0.0 velocity=0.0
- added joint Cube7_Cube14: type revolute, parent Cube7, child Cube14, origin xyz=0.33345319835012854 0.0 0.0 rpy=0 0 0, axis 0 1 0, limit lower=-3.14159 upper=3.14159 effort=0.0 velocity=0.0
- added joint Cube8_Cube9: type revolute, parent Cube8, child Cube9, origin xyz=0.0 -0.33485684809829114 -0.5469322503309809 rpy=0 0 0, axis 0 1 0, limit lower=-3.14159 upper=3.14159 effort=0.0 velocity=0.0
- joint Cube0_Cube1: origin xyz=0.0 -0.5662027639397147 3 rpy=0 0 0 -> xyz=0.0 -0.5749689440638529 3 rpy=0 0 0
- joint Cube0_Cube5: origin xyz=0.2845775799984116 0.0 3 rpy=0 0 0 -> xyz=0.0 0.5749689440638529 3 rpy=0 0 0
- joint Cube11_Cube12: origin xyz=0.0 0.0 -0.20079505147913354 rpy=0 0 0 -> xyz=0.0 0.19763344451753292 -0.17520276775536622 rpy=0 0 0
- joint Cube1_Cube2: origin xyz=0.0 -0.2074229003388439 -0.16642357061021806 rpy=0 0 0 -> xyz=0.0 -0.7880995429068027 0.0 rpy=0 0 0
- joint Cube2_Cube3: origin xyz=0.0 0.0 -0.2455740320331536 rpy=0 0 0 -> xyz=0.0 -0.17891535260447497 -0.1573833804840307 rpy=0 0 0
- joint Cube5_Cube6: origin xyz=0.0 -0.4811110773447532 0.0 rpy=0 0 0 -> xyz=0.0 0.20387926084840882 0.0 rpy=0 0 0
- joint Cube7_Cube8: origin xyz=0.0 -0.23171931050946817 -0.18576232255057484 rpy=0 0 0 -> xyz=0.16672659917506427 -0.5097602571485862 0.0 rpy=0 0 0
- joint Cube9_Cube10: origin xyz=0.0 0.20915522185902638 0.0 rpy=0 0 0 -> xyz=0.0 0.0 -0.43865901717092065 rpy=0 0 0
