Commit message: sped up snakes video

File: body.urdf (robot description, URDF)
Before this commit: robot robot, 15 links, 14 joints
Links:
- removed link Cube10
- removed link Cube11
- removed link Cube12
- removed link Cube13
- removed link Cube14
- removed link Cube7
- removed link Cube8
- removed link Cube9
- link Cube0: geometry collision box size=0.2708690656106623 0.8097915477163535 1.477676169791921; visual box size=0.2708690656106623 0.8097915477163535 1.477676169791921
- link Cube1: geometry collision box size=0.24502885576298045 0.35081176282144994 1.074629089984777; visual box size=0.24502885576298045 0.35081176282144994 1.074629089984777
- link Cube2: geometry collision box size=0.23973667168073529 0.22817042988525554 0.3676774070821345; visual box size=0.23973667168073529 0.22817042988525554 0.3676774070821345
- link Cube3: geometry collision box size=0.20105800404014323 0.21230492070720988 0.2469586394726287; visual box size=0.20105800404014323 0.21230492070720988 0.2469586394726287
- link Cube4: geometry collision box size=0.20019219040988445 0.20591994841452427 0.24479482030582733; visual box size=0.20019219040988445 0.20591994841452427 0.24479482030582733
- link Cube5: geometry collision box size=0.20013086451897838 0.20171375407342557 0.22514630675675068; visual box size=0.20013086451897838 0.20171375407342557 0.22514630675675068
- link Cube6: geometry collision box size=0.6371931266046219 0.33463990325065684 0.7257770255288258; visual box size=0.6371931266046219 0.33463990325065684 0.7257770255288258
Joints:
- removed joint Cube0_Cube5
- removed joint Cube0_Cube7
- removed joint Cube11_Cube12
- removed joint Cube12_Cube13
- removed joint Cube2_Cube3
- removed joint Cube5_Cube6
- removed joint Cube7_Cube11
- removed joint Cube7_Cube14
- removed joint Cube7_Cube8
- removed joint Cube8_Cube9
- removed joint Cube9_Cube10
- added joint Cube0_Cube3: type revolute, parent Cube0, child Cube3, origin xyz=0.0 0.40489577385817677 3 rpy=0 0 0, axis 0 1 0, limit lower=-3.14159 upper=3.14159 effort=0.0 velocity=0.0
- added joint Cube0_Cube6: type revolute, parent Cube0, child Cube6, origin xyz=0.13543453280533116 0.0 3 rpy=0 0 0, axis 0 1 0, limit lower=-3.14159 upper=3.14159 effort=0.0 velocity=0.0
- added joint Cube4_Cube5: type revolute, parent Cube4, child Cube5, origin xyz=0.0 0.20591994841452427 0.0 rpy=0 0 0, axis 0 1 0, limit lower=-3.14159 upper=3.14159 effort=0.0 velocity=0.0
- joint Cube0_Cube1: origin xyz=0.0 -0.5749689440638529 3 rpy=0 0 0 -> xyz=0.0 -0.40489577385817677 3 rpy=0 0 0
- joint Cube1_Cube2: origin xyz=0.0 -0.7880995429068027 0.0 rpy=0 0 0 -> xyz=0.0 -0.35081176282144994 0.0 rpy=0 0 0
- joint Cube3_Cube4: origin xyz=0.0 -0.1022692090072913 -0.12475577792441286 rpy=0 0 0 -> xyz=0.0 0.21230492070720988 0.0 rpy=0 0 0

Commit message: creating new branch

File: body.urdf (robot description, URDF)
Before this commit: robot robot, 7 links, 6 joints
Links:
- added link Cube10, mass 1; collision box size=0.6212206632618614 1.4179685484635511 1.1547591136457607; visual box size=0.6212206632618614 1.4179685484635511 1.1547591136457607
- added link Cube11, mass 1; collision box size=0.27780385196931034 0.6108624483865825 1.0640217266446255; visual box size=0.27780385196931034 0.6108624483865825 1.0640217266446255
- added link Cube12, mass 1; collision box size=0.23932044667938676 0.5966669129651174 0.8903902495175293; visual box size=0.23932044667938676 0.5966669129651174 0.8903902495175293
- added link Cube13, mass 1; collision box size=0.21905863813412382 0.37280402480139285 0.48502560807166006; visual box size=0.21905863813412382 0.37280402480139285 0.48502560807166006
- added link Cube14, mass 1; collision box size=0.5224948182091756 1.083169459367129 1.3895074880943787; visual box size=0.5224948182091756 1.083169459367129 1.3895074880943787
- added link Cube15, mass 1; collision box size=0.2672954720131415 0.6176325236704788 0.2734941864928033; visual box size=0.2672954720131415 0.6176325236704788 0.2734941864928033
- added link Cube16, mass 1; collision box size=0.24361657548372342 0.308596943464405 0.21293660857031513; visual box size=0.24361657548372342 0.308596943464405 0.21293660857031513
- added link Cube17, mass 1; collision box size=0.2245358219191934 0.2310131237003245 0.20505382485999066; visual box size=0.2245358219191934 0.2310131237003245 0.20505382485999066
- added link Cube18, mass 1; collision box size=0.22144238656997256 0.2174849998777975 0.2027680421825774; visual box size=0.22144238656997256 0.2174849998777975 0.2027680421825774
- added link Cube19, mass 1; collision box size=0.20217415266835767 0.20148254109920516 0.20017591591335396; visual box size=0.20217415266835767 0.20148254109920516 0.20017591591335396
- added link Cube20, mass 1; collision box size=0.20018434306381502 0.2013312176148146 0.20010155369690924; visual box size=0.20018434306381502 0.2013312176148146 0.20010155369690924
- added link Cube21, mass 1; collision box size=0.20015722178190706 0.20038349277233775 0.20006382216228183; visual box size=0.20015722178190706 0.20038349277233775 0.20006382216228183
- added link Cube22, mass 1; collision box size=0.20005897171143308 0.20023444192759474 0.2000257136258382; visual box size=0.20005897171143308 0.20023444192759474 0.2000257136258382
- added link Cube23, mass 1; collision box size=0.2000115321098065 0.20005502350467622 0.20000612771823906; visual box size=0.2000115321098065 0.20005502350467622 0.20000612771823906
- added link Cube24, mass 1; collision box size=0.46587689283775124 1.3592814134152598 0.44662948007117265; visual box size=0.46587689283775124 1.3592814134152598 0.44662948007117265
- added link Cube25, mass 1; collision box size=0.22348186382209628 1.0561312379773624 0.3612393536974212; visual box size=0.22348186382209628 1.0561312379773624 0.3612393536974212
- added link Cube26, mass 1; collision box size=0.21837162608595564 1.0328119022604838 0.2939478075519693; visual box size=0.21837162608595564 1.0328119022604838 0.2939478075519693
- added link Cube27, mass 1; collision box size=0.20981604582352084 0.9216451306497997 0.2520168581322678; visual box size=0.20981604582352084 0.9216451306497997 0.2520168581322678
- added link Cube28, mass 1; collision box size=0.20043943132849582 0.23219218975012548 0.2112832733348609; visual box size=0.20043943132849582 0.23219218975012548 0.2112832733348609
- added link Cube29, mass 1; collision box size=1.1552858725517998 0.7558986089816284 0.8095019299429116; visual box size=1.1552858725517998 0.7558986089816284 0.8095019299429116
- added link Cube7, mass 1; collision box size=0.23187088481823906 0.20094912463871037 0.20081681035149088; visual box size=0.23187088481823906 0.20094912463871037 0.20081681035149088
- added link Cube8, mass 1; collision box size=0.2190554749313029 0.20062413698411324 0.20065254626178328; visual box size=0.2190554749313029 0.20062413698411324 0.20065254626178328
- added link Cube9, mass 1; collision box size=0.2128595483990657 0.20006020304656394 0.2003801548010991; visual box size=0.2128595483990657 0.20006020304656394 0.2003801548010991
- link Cube0: geometry collision box size=1.2682994739163163 1.4233887778146372 0.8498320258026599; visual box size=1.2682994739163163 1.4233887778146372 0.8498320258026599
- link Cube1: geometry collision box size=0.5559921551143994 0.9690210703093876 0.34377714203353293; visual box size=0.5559921551143994 0.9690210703093876 0.34377714203353293
- link Cube2: geometry collision box size=0.30747057049766435 0.41971848716031573 0.25151090431794565; visual box size=0.30747057049766435 0.41971848716031573 0.25151090431794565
- link Cube3: geometry collision box size=0.2903378664849294 0.3437221093945361 0.22043319102189793; visual box size=0.2903378664849294 0.3437221093945361 0.22043319102189793
- link Cube4: geometry collision box size=0.2558004880727475 0.20197799816288894 0.21414757738682266; visual box size=0.2558004880727475 0.20197799816288894 0.21414757738682266
- link Cube5: geometry collision box size=0.2541707402491622 0.2014817811404633 0.21368841916039857; visual box size=0.2541707402491622 0.2014817811404633 0.21368841916039857
- link Cube6: geometry collision box size=0.24296914517727772 0.20096687631244034 0.21356401780061585; visual box size=0.24296914517727772 0.20096687631244034 0.21356401780061585
Joints:
- removed joint Cube0_Cube3
- added joint Cube0_Cube10: type revolute, parent Cube0, child Cube10, origin xyz=0.6341497369581581 0.0 3 rpy=0 0 0, axis 0 1 0, limit lower=-3.14159 upper=3.14159 effort=0.0 velocity=0.0
- added joint Cube10_Cube11: type revolute, parent Cube10, child Cube11, origin xyz=0.3106103316309307 -0.7089842742317756 0.0 rpy=0 0 0, axis 0 1 0, limit lower=-3.14159 upper=3.14159 effort=0.0 velocity=0.0
- added joint Cube10_Cube13: type revolute, parent Cube10, child Cube13, origin xyz=-0.3106103316309307 0.7089842742317756 0.0 rpy=0 0 0, axis 0 1 0, limit lower=-3.14159 upper=3.14159 effort=0.0 velocity=0.0
- added joint Cube10_Cube14: type revolute, parent Cube10, child Cube14, origin xyz=0.6212206632618614 0.0 0.0 rpy=0 0 0, axis 0 1 0, limit lower=-3.14159 upper=3.14159 effort=0.0 velocity=0.0
- added joint Cube11_Cube12: type revolute, parent Cube11, child Cube12, origin xyz=0.0 -0.3054312241932913 -0.5320108633223127 rpy=0 0 0, axis 0 1 0, limit lower=-3.14159 upper=3.14159 effort=0.0 velocity=0.0
- added joint Cube14_Cube15: type revolute, parent Cube14, child Cube15, origin xyz=0.2612474091045878 -0.5415847296835645 0.0 rpy=0 0 0, axis 0 1 0, limit lower=-3.14159 upper=3.14159 effort=0.0 velocity=0.0
- added joint Cube14_Cube20: type revolute, parent Cube14, child Cube20, origin xyz=-0.2612474091045878 0.5415847296835645 0.0 rpy=0 0 0, axis 0 1 0, limit lower=-3.14159 upper=3.14159 effort=0.0 velocity=0.0
- added joint Cube14_Cube24: type revolute, parent Cube14, child Cube24, origin xyz=0.5224948182091756 0.0 0.0 rpy=0 0 0, axis 0 1 0, limit lower=-3.14159 upper=3.14159 effort=0.0 velocity=0.0
- added joint Cube15_Cube16: type revolute, parent Cube15, child Cube16, origin xyz=0.0 -0.3088162618352394 -0.13674709324640166 rpy=0 0 0, axis 0 1 0, limit lower=-3.14159 upper=3.14159 effort=0.0 velocity=0.0
- added joint Cube16_Cube17: type revolute, parent Cube16, child Cube17, origin xyz=0.0 0.0 -0.21293660857031513 rpy=0 0 0, axis 0 1 0, limit lower=-3.14159 upper=3.14159 effort=0.0 velocity=0.0
- added joint Cube17_Cube18: type revolute, parent Cube17, child Cube18, origin xyz=0.0 -0.11550656185016225 -0.10252691242999533 rpy=0 0 0, axis 0 1 0, limit lower=-3.14159 upper=3.14159 effort=0.0 velocity=0.0
- added joint Cube18_Cube19: type revolute, parent Cube18, child Cube19, origin xyz=0.0 -0.10874249993889876 -0.1013840210912887 rpy=0 0 0, axis 0 1 0, limit lower=-3.14159 upper=3.14159 effort=0.0 velocity=0.0
- added joint Cube20_Cube21: type revolute, parent Cube20, child Cube21, origin xyz=0.0 0.1006656088074073 -0.10005077684845462 rpy=0 0 0, axis 0 1 0, limit lower=-3.14159 upper=3.14159 effort=0.0 velocity=0.0
- added joint Cube21_Cube22: type revolute, parent Cube21, child Cube22, origin xyz=0.0 0.10019174638616887 -0.10003191108114091 rpy=0 0 0, axis 0 1 0, limit lower=-3.14159 upper=3.14159 effort=0.0 velocity=0.0
- added joint Cube22_Cube23: type revolute, parent Cube22, child Cube23, origin xyz=0.0 0.10011722096379737 -0.1000128568129191 rpy=0 0 0, axis 0 1 0, limit lower=-3.14159 upper=3.14159 effort=0.0 velocity=0.0
- added joint Cube24_Cube25: type revolute, parent Cube24, child Cube25, origin xyz=0.23293844641887562 -0.6796407067076299 0.0 rpy=0 0 0, axis 0 1 0, limit lower=-3.14159 upper=3.14159 effort=0.0 velocity=0.0
- added joint Cube24_Cube26: type revolute, parent Cube24, child Cube26, origin xyz=-0.23293844641887562 0.6796407067076299 0.0 rpy=0 0 0, axis 0 1 0, limit lower=-3.14159 upper=3.14159 effort=0.0 velocity=0.0
- added joint Cube24_Cube29: type revolute, parent Cube24, child Cube29, origin xyz=0.46587689283775124 0.0 0.0 rpy=0 0 0, axis 0 1 0, limit lower=-3.14159 upper=3.14159 effort=0.0 velocity=0.0
- added joint Cube26_Cube27: type revolute, parent Cube26, child Cube27, origin xyz=0.0 0.5164059511302419 -0.14697390377598465 rpy=0 0 0, axis 0 1 0, limit lower=-3.14159 upper=3.14159 effort=0.0 velocity=0.0
- added joint Cube27_Cube28: type revolute, parent Cube27, child Cube28, origin xyz=0.0 0.0 -0.2520168581322678 rpy=0 0 0, axis 0 1 0, limit lower=-3.14159 upper=3.14159 effort=0.0 velocity=0.0
- added joint Cube2_Cube3: type revolute, parent Cube2, child Cube3, origin xyz=0.0 -0.41971848716031573 0.0 rpy=0 0 0, axis 0 1 0, limit lower=-3.14159 upper=3.14159 effort=0.0 velocity=0.0
- added joint Cube6_Cube7: type revolute, parent Cube6, child Cube7, origin xyz=0.0 0.10048343815622017 -0.10678200890030792 rpy=0 0 0, axis 0 1 0, limit lower=-3.14159 upper=3.14159 effort=0.0 velocity=0.0
- added joint Cube7_Cube8: type revolute, parent Cube7, child Cube8, origin xyz=0.0 0.0 -0.20081681035149088 rpy=0 0 0, axis 0 1 0, limit lower=-3.14159 upper=3.14159 effort=0.0 velocity=0.0
- added joint Cube8_Cube9: type revolute, parent Cube8, child Cube9, origin xyz=0.0 0.10031206849205662 -0.10032627313089164 rpy=0 0 0, axis 0 1 0, limit lower=-3.14159 upper=3.14159 effort=0.0 velocity=0.0
- joint Cube0_Cube1: origin xyz=0.0 -0.40489577385817677 3 rpy=0 0 0 -> xyz=0.0 -0.7116943889073186 3 rpy=0 0 0
- joint Cube0_Cube6: origin xyz=0.13543453280533116 0.0 3 rpy=0 0 0 -> xyz=0.0 0.7116943889073186 3 rpy=0 0 0
- joint Cube1_Cube2: origin xyz=0.0 -0.35081176282144994 0.0 rpy=0 0 0 -> xyz=0.0 -0.9690210703093876 0.0 rpy=0 0 0
- joint Cube3_Cube4: origin xyz=0.0 0.21230492070720988 0.0 rpy=0 0 0 -> xyz=0.0 -0.17186105469726806 -0.11021659551094896 rpy=0 0 0
- joint Cube4_Cube5: origin xyz=0.0 0.20591994841452427 0.0 rpy=0 0 0 -> xyz=0.0 -0.10098899908144447 -0.10707378869341133 rpy=0 0 0
