Commit message: generates different bodies for parents and kids, not need to make it evolve properly

File: body.urdf (robot description, URDF)
Before this commit: robot robot, 9 links, 8 joints
Links:
- removed link BackLeg
- removed link BackLowerLeg
- removed link FrontLeg
- removed link FrontLowerLeg
- removed link LeftLeg
- removed link LeftLowerLeg
- removed link RightLeg
- removed link RightLowerLeg
- removed link Torso
- added link Cube0, mass 1; collision box size=1.3156311747116187 1.2642622579956297 0.5778316993451812; visual box size=1.3156311747116187 1.2642622579956297 0.5778316993451812
- added link Cube1, mass 1; collision box size=0.5882543314292539 0.5713531035075314 0.4741635147651718; visual box size=0.5882543314292539 0.5713531035075314 0.4741635147651718
- added link Cube10, mass 1; collision box size=0.2225285016918925 0.559576045492486 0.6409064736379848; visual box size=0.2225285016918925 0.559576045492486 0.6409064736379848
- added link Cube11, mass 1; collision box size=0.20584173470066322 0.5556169549154015 0.4889551051770601; visual box size=0.20584173470066322 0.5556169549154015 0.4889551051770601
- added link Cube12, mass 1; collision box size=0.20137163343554162 0.3336138606274861 0.48297716402464747; visual box size=0.20137163343554162 0.3336138606274861 0.48297716402464747
- added link Cube13, mass 1; collision box size=0.5389327499859571 1.098679731800155 0.9355057643930902; visual box size=0.5389327499859571 1.098679731800155 0.9355057643930902
- added link Cube14, mass 1; collision box size=0.33984781752440685 0.7565975330499748 0.2882646587142594; visual box size=0.33984781752440685 0.7565975330499748 0.2882646587142594
- added link Cube15, mass 1; collision box size=0.3296447720105484 0.6152792757058434 0.20019254648773013; visual box size=0.3296447720105484 0.6152792757058434 0.20019254648773013
- added link Cube16, mass 1; collision box size=0.32504521863092206 0.4659974129631553 0.20015557782321317; visual box size=0.32504521863092206 0.4659974129631553 0.20015557782321317
- added link Cube17, mass 1; collision box size=1.0865484683184499 0.6951248691272618 0.5008232380734368; visual box size=1.0865484683184499 0.6951248691272618 0.5008232380734368
- added link Cube18, mass 1; collision box size=0.2349753520016419 0.2487835470297844 0.49661733931899205; visual box size=0.2349753520016419 0.2487835470297844 0.49661733931899205
- added link Cube19, mass 1; collision box size=0.22700420568143442 0.24497344617406352 0.3899046634482446; visual box size=0.22700420568143442 0.24497344617406352 0.3899046634482446
- added link Cube2, mass 1; collision box size=0.6155685525158685 0.4763963452091138 0.37306473419187935; visual box size=0.6155685525158685 0.4763963452091138 0.37306473419187935
- added link Cube20, mass 1; collision box size=0.21743209992863782 0.21976595393097623 0.2110578111551501; visual box size=0.21743209992863782 0.21976595393097623 0.2110578111551501
- added link Cube21, mass 1; collision box size=0.2152922490926899 0.20284736377599466 0.20376374341525752; visual box size=0.2152922490926899 0.20284736377599466 0.20376374341525752
- added link Cube22, mass 1; collision box size=0.20706010558985813 0.20202924755183294 0.2010414135923192; visual box size=0.20706010558985813 0.20202924755183294 0.2010414135923192
- added link Cube23, mass 1; collision box size=1.2932691989751794 1.048875220982115 1.1755865365573794; visual box size=1.2932691989751794 1.048875220982115 1.1755865365573794
- added link Cube24, mass 1; collision box size=0.5030369737926663 0.559070906965139 0.5011270855448453; visual box size=0.5030369737926663 0.559070906965139 0.5011270855448453
- added link Cube25, mass 1; collision box size=0.3745516531726577 0.30833733185151285 0.2068025998394677; visual box size=0.3745516531726577 0.30833733185151285 0.2068025998394677
- added link Cube26, mass 1; collision box size=0.3336612013377185 0.20520849691066487 0.20277898368732591; visual box size=0.3336612013377185 0.20520849691066487 0.20277898368732591
- added link Cube27, mass 1; collision box size=0.25010098617624815 0.20146831084107863 0.20194137921371558; visual box size=0.25010098617624815 0.20146831084107863 0.20194137921371558
- added link Cube28, mass 1; collision box size=0.2081383697184711 0.2004043536119473 0.2001415927511121; visual box size=0.2081383697184711 0.2004043536119473 0.2001415927511121
- added link Cube29, mass 1; collision box size=0.20813457111960607 0.2000797147415559 0.20009086111958366; visual box size=0.20813457111960607 0.2000797147415559 0.20009086111958366
- added link Cube3, mass 1; collision box size=0.2553514782044186 0.4678804836540866 0.288787151429053; visual box size=0.2553514782044186 0.4678804836540866 0.288787151429053
- added link Cube30, mass 1; collision box size=0.4335529106612772 1.0603335603401352 0.8890443898590781; visual box size=0.4335529106612772 1.0603335603401352 0.8890443898590781
- added link Cube4, mass 1; collision box size=0.21349623028618528 0.3827227149409609 0.2701880059431896; visual box size=0.21349623028618528 0.3827227149409609 0.2701880059431896
- added link Cube5, mass 1; collision box size=0.21097212839688487 0.2816229158150143 0.2664384171100396; visual box size=0.21097212839688487 0.2816229158150143 0.2664384171100396
- added link Cube6, mass 1; collision box size=0.20130501429016615 0.28036359918340426 0.24735376683847204; visual box size=0.20130501429016615 0.28036359918340426 0.24735376683847204
- added link Cube7, mass 1; collision box size=0.20109779780775852 0.25390832022893606 0.24143912004632576; visual box size=0.20109779780775852 0.25390832022893606 0.24143912004632576
- added link Cube8, mass 1; collision box size=0.200073061998849 0.22830652817371822 0.20567663977466005; visual box size=0.200073061998849 0.22830652817371822 0.20567663977466005
- added link Cube9, mass 1; collision box size=0.6087754581587423 1.274379612463797 1.2484804216305214; visual box size=0.6087754581587423 1.274379612463797 1.2484804216305214
Joints:
- removed joint Torso_BackLeg
- removed joint Torso_BackLowerLeg
- removed joint Torso_FrontLeg
- removed joint Torso_FrontLowerLeg
- removed joint Torso_LeftLeg
- removed joint Torso_LeftLowerLeg
- removed joint Torso_RightLeg
- removed joint Torso_RightLowerLeg
- added joint Cube0_Cube1: type revolute, parent Cube0, child Cube1, origin xyz=0.0 -0.6321311289978149 3 rpy=0 0 0, axis 0 1 0, limit lower=-3.14159 upper=3.14159 effort=0.0 velocity=0.0
- added joint Cube0_Cube2: type revolute, parent Cube0, child Cube2, origin xyz=0.6578155873558094 0.0 3 rpy=0 0 0, axis 0 1 0, limit lower=-3.14159 upper=3.14159 effort=0.0 velocity=0.0
- added joint Cube11_Cube12: type revolute, parent Cube11, child Cube12, origin xyz=0.0 0.27780847745770076 -0.24447755258853004 rpy=0 0 0, axis 0 1 0, limit lower=-3.14159 upper=3.14159 effort=0.0 velocity=0.0
- added joint Cube13_Cube14: type revolute, parent Cube13, child Cube14, origin xyz=0.26946637499297854 -0.5493398659000776 0.0 rpy=0 0 0, axis 0 1 0, limit lower=-3.14159 upper=3.14159 effort=0.0 velocity=0.0
- added joint Cube13_Cube16: type revolute, parent Cube13, child Cube16, origin xyz=-0.26946637499297854 0.5493398659000776 0.0 rpy=0 0 0, axis 0 1 0, limit lower=-3.14159 upper=3.14159 effort=0.0 velocity=0.0
- added joint Cube13_Cube17: type revolute, parent Cube13, child Cube17, origin xyz=0.5389327499859571 0.0 0.0 rpy=0 0 0, axis 0 1 0, limit lower=-3.14159 upper=3.14159 effort=0.0 velocity=0.0
- added joint Cube14_Cube15: type revolute, parent Cube14, child Cube15, origin xyz=0.0 -0.3782987665249874 -0.1441323293571297 rpy=0 0 0, axis 0 1 0, limit lower=-3.14159 upper=3.14159 effort=0.0 velocity=0.0
- added joint Cube17_Cube18: type revolute, parent Cube17, child Cube18, origin xyz=0.5432742341592249 -0.3475624345636309 0.0 rpy=0 0 0, axis 0 1 0, limit lower=-3.14159 upper=3.14159 effort=0.0 velocity=0.0
- added joint Cube17_Cube20: type revolute, parent Cube17, child Cube20, origin xyz=-0.5432742341592249 0.3475624345636309 0.0 rpy=0 0 0, axis 0 1 0, limit lower=-3.14159 upper=3.14159 effort=0.0 velocity=0.0
- added joint Cube17_Cube23: type revolute, parent Cube17, child Cube23, origin xyz=1.0865484683184499 0.0 0.0 rpy=0 0 0, axis 0 1 0, limit lower=-3.14159 upper=3.14159 effort=0.0 velocity=0.0
- added joint Cube18_Cube19: type revolute, parent Cube18, child Cube19, origin xyz=0.0 -0.2487835470297844 0.0 rpy=0 0 0, axis 0 1 0, limit lower=-3.14159 upper=3.14159 effort=0.0 velocity=0.0
- added joint Cube20_Cube21: type revolute, parent Cube20, child Cube21, origin xyz=0.0 0.21976595393097623 0.0 rpy=0 0 0, axis 0 1 0, limit lower=-3.14159 upper=3.14159 effort=0.0 velocity=0.0
- added joint Cube21_Cube22: type revolute, parent Cube21, child Cube22, origin xyz=0.0 0.20284736377599466 0.0 rpy=0 0 0, axis 0 1 0, limit lower=-3.14159 upper=3.14159 effort=0.0 velocity=0.0
- added joint Cube23_Cube24: type revolute, parent Cube23, child Cube24, origin xyz=0.6466345994875897 -0.5244376104910575 0.0 rpy=0 0 0, axis 0 1 0, limit lower=-3.14159 upper=3.14159 effort=0.0 velocity=0.0
- added joint Cube23_Cube25: type revolute, parent Cube23, child Cube25, origin xyz=-0.6466345994875897 0.5244376104910575 0.0 rpy=0 0 0, axis 0 1 0, limit lower=-3.14159 upper=3.14159 effort=0.0 velocity=0.0
- added joint Cube23_Cube30: type revolute, parent Cube23, child Cube30, origin xyz=1.2932691989751794 0.0 0.0 rpy=0 0 0, axis 0 1 0, limit lower=-3.14159 upper=3.14159 effort=0.0 velocity=0.0
- added joint Cube25_Cube26: type revolute, parent Cube25, child Cube26, origin xyz=0.0 0.15416866592575643 -0.10340129991973385 rpy=0 0 0, axis 0 1 0, limit lower=-3.14159 upper=3.14159 effort=0.0 velocity=0.0
- added joint Cube26_Cube27: type revolute, parent Cube26, child Cube27, origin xyz=0.0 0.0 -0.20277898368732591 rpy=0 0 0, axis 0 1 0, limit lower=-3.14159 upper=3.14159 effort=0.0 velocity=0.0
- added joint Cube27_Cube28: type revolute, parent Cube27, child Cube28, origin xyz=0.0 0.10073415542053932 -0.10097068960685779 rpy=0 0 0, axis 0 1 0, limit lower=-3.14159 upper=3.14159 effort=0.0 velocity=0.0
- added joint Cube28_Cube29: type revolute, parent Cube28, child Cube29, origin xyz=0.0 0.2004043536119473 0.0 rpy=0 0 0, axis 0 1 0, limit lower=-3.14159 upper=3.14159 effort=0.0 velocity=0.0
- added joint Cube2_Cube3: type revolute, parent Cube2, child Cube3, origin xyz=0.30778427625793425 -0.2381981726045569 0.0 rpy=0 0 0, axis 0 1 0, limit lower=-3.14159 upper=3.14159 effort=0.0 velocity=0.0
- added joint Cube2_Cube7: type revolute, parent Cube2, child Cube7, origin xyz=-0.30778427625793425 0.2381981726045569 0.0 rpy=0 0 0, axis 0 1 0, limit lower=-3.14159 upper=3.14159 effort=0.0 velocity=0.0
- added joint Cube2_Cube9: type revolute, parent Cube2, child Cube9, origin xyz=0.6155685525158685 0.0 0.0 rpy=0 0 0, axis 0 1 0, limit lower=-3.14159 upper=3.14159 effort=0.0 velocity=0.0
- added joint Cube3_Cube4: type revolute, parent Cube3, child Cube4, origin xyz=0.0 -0.4678804836540866 0.0 rpy=0 0 0, axis 0 1 0, limit lower=-3.14159 upper=3.14159 effort=0.0 velocity=0.0
- added joint Cube4_Cube5: type revolute, parent Cube4, child Cube5, origin xyz=0.0 -0.19136135747048044 -0.1350940029715948 rpy=0 0 0, axis 0 1 0, limit lower=-3.14159 upper=3.14159 effort=0.0 velocity=0.0
- added joint Cube5_Cube6: type revolute, parent Cube5, child Cube6, origin xyz=0.0 0.0 -0.2664384171100396 rpy=0 0 0, axis 0 1 0, limit lower=-3.14159 upper=3.14159 effort=0.0 velocity=0.0
- added joint Cube7_Cube8: type revolute, parent Cube7, child Cube8, origin xyz=0.0 0.25390832022893606 0.0 rpy=0 0 0, axis 0 1 0, limit lower=-3.14159 upper=3.14159 effort=0.0 velocity=0.0
- added joint Cube9_Cube10: type revolute, parent Cube9, child Cube10, origin xyz=0.30438772907937117 -0.6371898062318985 0.0 rpy=0 0 0, axis 0 1 0, limit lower=-3.14159 upper=3.14159 effort=0.0 velocity=0.0
- added joint Cube9_Cube11: type revolute, parent Cube9, child Cube11, origin xyz=-0.30438772907937117 0.6371898062318985 0.0 rpy=0 0 0, axis 0 1 0, limit lower=-3.14159 upper=3.14159 effort=0.0 velocity=0.0
- added joint Cube9_Cube13: type revolute, parent Cube9, child Cube13, origin xyz=0.6087754581587423 0.0 0.0 rpy=0 0 0, axis 0 1 0, limit lower=-3.14159 upper=3.14159 effort=0.0 velocity=0.0
